File: sortirovka.brd (EAGLE design)
At the start: 86.7 x 86.7 mm, 71 parts, among them IC1 DS1307Z, IC3 LM1117IMPX-3.3, U1 MAX3485CSA, X1 PI3-CON, X10 MKDSN1,5/3-5,08, X3 MKDSN1,5/4-5,08, X4 MKDSN1,5/2-5,08, X5 22-23-2021, X6 22-23-2051, X7 22-23-2041, X8 22-23-2051, X9 MKDSN1,5/7-5,08

Commit message: wip
Parts:
- added Q1: (no value), MyLib:SOT23-6
Connections:
- new net N$48: Q1.1, Q1.2, Q1.5, Q1.6, X5.1
- net GND: now also Q1.3
- net PW: now also Q1.4; no longer X5.1
Routing:
- net N$48: track 0.00 -> 12.0 mm
- net PW: track 71.8 -> 61.3 mm
- net N$19: track 0.00 -> 2.98 mm
- net N$29: track 0.00 -> 2.66 mm
- net N$18: track 0.00 -> 2.60 mm
- net N$4: track 17.7 -> 16.5 mm
Changed lines of the file:
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@@
 <element name="C4" library="rcl" package="E3,5-8" value="" x="46.1645" y="9.4615" rot="R270"/>
 <element name="C6" library="rcl" package="C0805" value="0.1" x="52.197" y="1.4605" rot="MR270"/>
+<element name="Q1" library="MyLib" package="SOT23-6" value="" x="70.739" y="46.736" rot="MR0"/>
 </elements>
 <signals>
@@
 <contactref element="C5" pad="2"/>
 <contactref element="IC3" pad="1"/>
-<contactref element="X5" pad="2"/>
 <contactref element="C1" pad="-"/>
 <contactref element="C2" pad="-"/>
@@
 <wire x1="0.635" y1="63.0555" x2="0.3175" y2="62.738" width="0.4064" layer="16"/>
 <wire x1="0.3175" y1="62.738" x2="0.3175" y2="61.1505" width="0.4064" layer="16"/>
+<contactref element="X5" pad="2"/>
+<contactref element="Q1" pad="3"/>
 <wire x1="46.7233" y1="61.7474" x2="44.1833" y2="56.6674" width="0" layer="19" extent="1-1"/>
 </signal>
@@
 <contactref element="R18" pad="2"/>
 <contactref element="U$3" pad="1"/>
-<contactref element="U1" pad="7"/>
-<wire x1="60.96" y1="73.279" x2="59.823" y2="73.279" width="0.4064" layer="16"/>
 <wire x1="71.3715" y1="72.0885" x2="71.3715" y2="71.1175" width="0.4064" layer="16"/>
 <wire x1="64.262" y1="69.977" x2="60.96" y2="73.279" width="0.4064" layer="16"/>
@@
 <wire x1="64.643" y1="68.326" x2="64.643" y2="69.977" width="0.4064" layer="16"/>
 <wire x1="64.643" y1="69.977" x2="64.7065" y2="69.977" width="0.4064" layer="16"/>
+<contactref element="U1" pad="7"/>
+<wire x1="59.823" y1="73.279" x2="60.96" y2="73.279" width="0" layer="19" extent="16-16"/>
 </signal>
 <signal name="SPI0">
@@
 <contactref element="OC8" pad="1"/>
 <wire x1="61.341" y1="21.661" x2="61.3435" y2="21.661" width="0.4064" layer="16"/>
-<wire x1="61.341" y1="21.661" x2="61.3385" y2="24.257" width="0" layer="19" extent="16-16"/>
+<wire x1="61.3385" y1="24.257" x2="61.3385" y2="21.661" width="0.4064" layer="16"/>
+<wire x1="61.3385" y1="21.661" x2="61.341" y2="21.661" width="0.4064" layer="16"/>
 </signal>
 <signal name="N$19">
@@
 <contactref element="OC9" pad="1"/>
 <wire x1="68.7705" y1="21.661" x2="68.773" y2="21.661" width="0.4064" layer="16"/>
-<wire x1="68.7705" y1="21.661" x2="68.7705" y2="24.6405" width="0" layer="19" extent="16-16"/>
+<wire x1="68.7705" y1="24.6405" x2="68.7705" y2="21.661" width="0.4064" layer="16"/>
 </signal>
 <signal name="N$29">
@@
 <contactref element="OC10" pad="1"/>
 <wire x1="75.819" y1="21.661" x2="75.8215" y2="21.661" width="0.4064" layer="16"/>
-<wire x1="75.819" y1="21.661" x2="75.819" y2="24.323" width="0" layer="19" extent="16-16"/>
+<wire x1="75.819" y1="24.323" x2="75.819" y2="21.661" width="0.4064" layer="16"/>
 </signal>
 <signal name="PW">
-<contactref element="X5" pad="1"/>
 <contactref element="IC3" pad="3"/>
 <contactref element="R14" pad="2"/>
-<contactref element="C2" pad="+"/>
 <contactref element="C3" pad="1"/>
 <wire x1="56.896" y1="77.4675" x2="56.896" y2="69.342" width="0.4064" layer="16"/>
@@
 <wire x1="55.7555" y1="54.2925" x2="54.458" y2="54.2925" width="0.4064" layer="16"/>
 <wire x1="54.458" y1="54.2925" x2="54.3945" y2="54.229" width="0.4064" layer="16"/>
-<wire x1="54.3945" y1="49.53" x2="54.3945" y2="50.165" width="0.8128" layer="16"/>
-<wire x1="54.3945" y1="50.165" x2="54.3945" y2="51.816" width="0.8128" layer="16"/>
-<wire x1="54.3945" y1="51.816" x2="54.3945" y2="54.229" width="0.8128" layer="16"/>
-<wire x1="55.626" y1="51.816" x2="54.3945" y2="51.816" width="0.8128" layer="16"/>
 <wire x1="56.896" y1="77.4675" x2="48.321" y2="77.4675" width="0.4064" layer="16"/>
 <wire x1="48.321" y1="77.4675" x2="47.1805" y2="76.327" width="0.4064" layer="16"/>
@@
 <wire x1="53.6575" y1="59.69" x2="54.3945" y2="58.953" width="0.4064" layer="16"/>
 <wire x1="54.3945" y1="58.953" x2="54.3945" y2="56.7815" width="0.4064" layer="16"/>
-<wire x1="79.1845" y1="48.006" x2="54.3945" y2="48.006" width="0.8128" layer="16"/>
-<wire x1="54.3945" y1="48.006" x2="54.3945" y2="49.53" width="0.8128" layer="16"/>
+<wire x1="54.3945" y1="48.006" x2="54.3945" y2="48.1965" width="0.8128" layer="16"/>
+<contactref element="C2" pad="+"/>
+<contactref element="Q1" pad="4"/>
+<wire x1="54.3945" y1="48.1965" x2="54.3945" y2="54.229" width="0.8128" layer="16"/>
+<wire x1="69.789" y1="48.036" x2="69.789" y2="48.1965" width="0.6096" layer="16"/>
+<wire x1="69.789" y1="48.1965" x2="54.3945" y2="48.1965" width="0.6096" layer="16"/>
+<wire x1="55.7555" y1="54.2925" x2="55.626" y2="51.816" width="0" layer="19" extent="16-16"/>
 </signal>
 <signal name="N$45">
@@
 <wire x1="9.9695" y1="53.5305" x2="9.9695" y2="51.181" width="0.4064" layer="16"/>
 </signal>
+<signal name="N$48">
+<contactref element="X5" pad="1"/>
+<contactref element="Q1" pad="1"/>
+<contactref element="Q1" pad="2"/>
+<contactref element="Q1" pad="5"/>
+<contactref element="Q1" pad="6"/>
+<wire x1="79.1845" y1="48.006" x2="79.1845" y2="48.036" width="0.8128" layer="16"/>
+<wire x1="79.1845" y1="48.036" x2="71.689" y2="48.036" width="0.8128" layer="16"/>
+<wire x1="70.739" y1="48.036" x2="71.689" y2="48.036" width="0.6096" layer="16"/>
+<wire x1="71.689" y1="48.036" x2="71.689" y2="45.436" width="0.6096" layer="16"/>
+<wire x1="71.689" y1="45.436" x2="70.739" y2="45.436" width="0.6096" layer="16"/>
+</signal>
 </signals>

Commit message: wip
Parts:
- removed R12, R13, R5, R6, R8, R9: 1k, rcl:R0805
- removed R14, R7: 0, rcl:R0805
- removed R16, R17: 15, rcl:0207/10
- removed R18, R19: 1k5, rcl:0207/10
- removed R20: 10, rcl:0207/10
- removed X10: MKDSN1,5/3-5,08, con-phoenix-508:MKDSN1,5/3-5,08
- added C11, C12: (no value), rcl:C0805
- added C13, C20: 10uF, rcl:C0805
- added C14, C16, C18, C19: 100nF, rcl:C0805
- added C15, C17: 10nF, rcl:C0805
- added D11: CDSOT23-SM712SOT23-R, MyLib:SOT23-R
- added D12, D13: DIODE1N4007, MyLib:SMA-DIODE
- added GDT1, GDT2: GDT-2031-XXT-SM, supressor:2031-XXT-SM
- added IC2: MEGA8-AI, atmel:TQFP32-08
- added IC4, IC5: PCF8574T, micro-philips:SO16W
- added IC6: MEGA32-A, atmel:TQFP44
- added JP1: (no value), pinhead:1X09/90
- added JP4: (no value), pinhead:2X03
- added L1, L2: (no value), rcl:L0402
- added OC11, OC12: (no value), MyLib:SFH6106
- added Q2: (no value), crystal:SM49
- added U$8: NSI45020AT1GSOD-123, MyLib:SOD123
- added Z1, Z2: TBU-CA, supressor:TBU-CA
- R1, R2, R3, R4: value 200 -> 50
- R15: value 120 -> 1k; device rcl:0207/10 -> rcl:R0805
- U$3: value NUP2105LSOT23-R -> NSI45020AT1GSOD-123; device MyLib:SOT23-R -> MyLib:SOD123
- U1: value MAX3485CSA -> ADM2587EBRWZ; device MyLib:SO08 -> Analog Devices_By_element14_Batch_1:SOIC127P1032X265-20N
- X1: value PI3-CON -> MKDSN1,5/3-5,08; device MyLib:RPI3 -> MyLib:MKDSN1,5/3-5,08
- moved C8 161.9 mm to (162.6, 66.5), flipped to the top
- moved C9 151.0 mm to (157.1, 38.0), flipped to the top
- moved X6 143.5 mm to (153.4, 73.3), flipped to the bottom
- moved X8 143.5 mm to (153.4, 65.6), flipped to the bottom
- moved G1 142.5 mm to (152.8, 45.1), flipped to the bottom
- moved Q5 139.4 mm to (151.3, 48.5), flipped to the top
- moved U$1 133.2 mm to (136.1, 16.1), flipped to the top
- moved OC1 132.0 mm to (135.5, 24.2), flipped to the top
- moved IC1 128.3 mm to (145.7, 56.2), flipped to the top
- moved R11 128.1 mm to (145.7, 51.3), flipped to the top
- moved D5 125.0 mm to (132.0, 9.40), flipped to the top
- moved C5 122.9 mm to (143.1, 47.1), flipped to the top
- moved U$2 119.5 mm to (129.3, 16.1), flipped to the top
- moved OC2 119.0 mm to (129.0, 24.3), flipped to the top
- moved R10 117.9 mm to (140.5, 51.4), flipped to the top
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Connections:
- removed net N$43: OC1.4, R5.2, X1.P$7
- new net +5V: JP4.2
- new net A: D11.1, U1.18, Z1.3
- new net AVCC: IC2.18, IC6.27
- new net B: D11.2, U1.17, Z2.3
- new net GND2: IC6.39
- new net INT-S: IC4.4, IC5.13
- new net INT0: IC2.32, IC4.13
- new net N$49: IC4.9, JP1.5
- new net N$50: IC4.7, JP1.6
- new net N$51: IC4.6, JP1.7
- new net N$52: IC4.5, JP1.9
- new net N$53: JP1.8, R15.1
- new net N$54: IC5.12, OC1.3
- new net N$55: IC5.11, OC2.3
- new net N$56: IC5.10, OC3.3
- new net N$57: IC5.9, OC4.3
- new net N$58: IC5.7, OC5.3
- new net PE: C13.2, C15.2, C16.2, D11.3, GDT1.1, GDT2.2, L2.2, U1.16, U1.20, X1.2
- new net R/W: IC2.12, U1.5, U1.6
- new net RESET: IC2.29, JP4.5
- new net RS2: IC2.1
- new net RXD: IC2.30, U1.4
- new net SCK: IC2.17, JP4.3
- new net SCL: IC1.6, IC2.28, IC4.14, IC5.14, R10.1, X7.3
- new net SDA: IC1.5, IC2.27, IC4.15, IC5.15, R11.1, X7.2
- new net TXD: IC2.31, U1.7
- new net VCC: C17.1, C18.1, C19.1, C20.1, IC2.4, IC2.6, IC6.5, U1.2, U1.8
- new net VCC1: IC6.17
- new net VCC2: IC6.38
- net +3V3: now also IC4.16, IC5.1, IC5.16, R15.2; no longer OC1.3, OC2.3, OC3.3, OC4.3, OC5.3, OC6.3, R19.2, R7.2, U1.8
- net GND: now also C11.2, C12.1, C17.2, C18.2, C19.2, C20.2, IC2.21, IC2.3, IC2.5, IC4.1, IC4.2, IC4.3, IC4.8, IC5.2, IC5.3, IC5.8, IC6.28, IC6.6, JP1.1, JP4.6, OC1.4, OC11.4, OC12.4, OC2.4, OC3.4, OC4.4, OC5.4, OC6.4, U1.1, U1.10, U1.3, U1.9; no longer R12.1, R13.1, R18.1, R20.2, R5.1, R6.1, R8.1, R9.1, U$3.3, U1.5, X1.P$14, X1.P$20, X1.P$25, X1.P$30, X1.P$34, X1.P$39, X1.P$6, X1.P$9
- net GND1: now also D12.A, D13.A, IC6.18, OC11.2, OC12.2
- net MISO: now also IC2.16, JP4.1; no longer X1.P$21
- net MOSI: now also IC2.15, JP4.4; no longer X1.P$19
- net N$1: now also GDT1.2, X1.1, Z1.1; no longer U1.4, X1.P$8
- net N$14: now also C11.1, IC2.8, Q2.1; no longer R7.1, X1.P$1, X1.P$17
- net N$2: now also GDT2.1, X1.3, Z2.1; no longer U1.1, X1.P$10
- net N$26: now also C12.2, IC2.7, Q2.2; no longer IC1.6, R10.1, X1.P$5, X7.3
- net N$27: now also D12.C, OC11.1, U$3.C; no longer IC1.5, R11.1, X1.P$3, X7.2
- net N$28: now also U$3.A; no longer R14.1, X1.P$2, X1.P$4
- net N$3: now also C13.1, C15.1, C16.1, L1.2, U1.19; no longer U1.2, U1.3, X1.P$12
- net N$34: now also D13.C, OC12.1, U$8.C; no longer OC6.4, R13.2, X1.P$37
- net N$39: now also U$8.A; no longer OC5.4, R12.2, X1.P$35
- net N$4: now also C14.2, L2.1, U1.11, U1.14; no longer R16.2, R18.2, U$3.1, U1.7
- net N$40: now also IC5.6, OC6.3; no longer OC4.4, R9.2, X1.P$33
- net N$41: now also IC5.5, OC11.3; no longer OC3.4, R8.2, X1.P$31
- net N$42: now also IC5.4, OC12.3; no longer OC2.4, R6.2, X1.P$29
- net N$45: now also IC4.12, JP1.2; no longer R15.2, R16.1, X10.2
- net N$46: now also IC4.11, JP1.3; no longer R15.1, R17.1, X10.1
- net N$47: now also IC4.10, JP1.4; no longer R17.2, R19.1, U$3.2, U1.6
- net N$5: now also C14.1, L1.1, U1.12; no longer R20.1, X10.3
- net N$6: now also IC2.23, R4.2; no longer R1.2, X1.P$40
- net N$7: now also IC2.24, R3.2; no longer R2.2, X1.P$38
- net N$8: now also IC2.25, R2.2; no longer R3.2, X1.P$36
- net N$9: now also IC2.26, R1.2; no longer R4.2, X1.P$32
- net PW: no longer R14.2
- net SPI0: no longer X1.P$24
- net SPI1: no longer X1.P$26
- net SPI_CLK: no longer X1.P$23
Routing:
- net GND: track 217.7 -> 63.3 mm, vias 12 -> 0
- net +3V3: track 262.8 -> 150.2 mm, vias 2 -> 1
- net SPI_CLK: track 74.3 -> 0.00 mm
- net N$26: track 69.0 -> 0.00 mm
- net N$27: track 65.8 -> 0.00 mm
- net MISO: track 72.8 -> 7.68 mm
- net MOSI: track 72.3 -> 7.68 mm
- net N$43: track 57.5 -> 0.00 mm, vias 2 -> 0
- net N$42: track 42.2 -> 0.00 mm
- net N$41: track 36.3 -> 0.00 mm
- net N$9: track 33.5 -> 0.00 mm
- net N$40: track 30.1 -> 0.00 mm
- net VCC: track 0.00 -> 25.9 mm
- net N$8: track 23.3 -> 0.00 mm
- net N$45: track 22.9 -> 0.00 mm
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- removed copper zone on layer 16, net GND
Other:
- board size 86.7 x 86.7 mm -> 168.4 x 86.7 mm
