File: sortirovka.brd (EAGLE design)
At the start: 168.4 x 86.7 mm, 87 parts, among them IC1 DS1307Z, IC2 MEGA8-AI, IC3 LM1117IMPX-3.3, IC4 PCF8574T, IC5 PCF8574T, IC6 MEGA32-A, U1 ADM2587EBRWZ, X1 MKDSN1,5/3-5,08, X3 MKDSN1,5/4-5,08, X4 MKDSN1,5/2-5,08, X5 22-23-2021, X6 22-23-2051, X7 22-23-2041, X8 22-23-2051, X9 MKDSN1,5/7-5,08

Commit message: main pars on the board
Parts:
- removed Q1: (no value), MyLib:SOT23-6
- removed X8: 22-23-2051, con-molex:22-23-2051
- added J1: ATTEND-MICROSD-112, sd-mmc:ATTEND-112
- added R12, R5, R6: 3.3k, rcl:M0805
- added R13: 100k, rcl:M0805
- added R7, R8, R9: 1.8k, rcl:M0805
- added U$10: 2X16LCDBOTH, MyLib:2X16LCDBOTH
- added U$9: W5100_MODULESMALL, MyLib:W5100_MODULE_1
- IC6: value MEGA32-A -> PCF8574T; device atmel:TQFP44 -> micro-philips:SO16W
- JP1: device pinhead:1X09/90 -> pinhead:1X09
- moved C7 150.7 mm to (0.57, 50.1)
- moved IC3 150.7 mm to (5.02, 40.7)
- moved C1 150.7 mm to (4.25, 46.9)
- moved C10 150.7 mm to (0.70, 58.3)
- moved C2 150.7 mm to (4.32, 32.6)
- moved C3 150.7 mm to (5.02, 35.1)
- moved X6 140.8 mm to (15.4, 45.2), flipped to the top
- moved C6 128.0 mm to (158.9, 6.92)
- moved C4 113.3 mm to (150.2, 10.4)
- moved X4 113.3 mm to (150.3, 1.52)
- moved C5 90.5 mm to (62.0, 87.4), turned to 180 degrees
- moved IC6 90.0 mm to (106.0, 61.0)
- moved Q5 78.7 mm to (75.1, 68.1), turned to 90 degrees
- moved IC1 72.5 mm to (73.2, 58.0), turned to 180 degrees
- moved C8 52.6 mm to (202.2, 32.0)
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Connections:
- removed net GND2: IC6.39
- removed net PW: C2.+, C3.1, IC3.3, Q1.4
- removed net SPI1: X8.4
- removed net VCC1: IC6.17
- removed net VCC2: IC6.38
- new net E_RESET: U$9.RESET
- new net E_SELECT: U$9.SS
- new net ID0: IC6.9, U$10.21, U$10.7
- new net ID1: IC6.10, U$10.22, U$10.8
- new net ID2: IC6.11, U$10.23, U$10.9
- new net ID3: IC6.12, U$10.10, U$10.24
- new net I_E: IC6.7, U$10.20, U$10.6
- new net I_RS: IC6.5, U$10.18, U$10.4
- new net I_RW: IC6.6, U$10.19, U$10.5
- new net N$43: J1.DAT3, R12.2, R9.1
- new net N$59: J1.CMD, R6.2, R8.1
- new net N$60: J1.CLK, R5.2, R7.1
- new net N$61: IC6.14
- new net N$73: U$10.17, U$10.3
- new net SD_DETECT: J1.CD, R13.1
- new net SD_SELECT: R9.2
- net +3V3: now also J1.VDD, R13.2; no longer IC1.8, IC4.16, IC5.1, IC5.16, R10.2, R11.2, R15.2, X7.1
- net +5V: now also C17.1, C18.1, C19.1, C2.+, C20.1, C3.1, IC1.8, IC3.3, IC4.16, IC5.1, IC5.16, IC6.16, IC6.2, R10.2, R11.2, R15.2, U$10.16, U$10.2, U$9.VCC, U1.2, U1.8, X5.1, X7.1
- net AVCC: no longer IC6.27
- net GND: now also IC6.1, IC6.3, IC6.8, J1.GND, J1.S1, J1.S2, J1.VSS, R12.1, R5.1, R6.1, U$10.1, U$10.15, U$9.GND@1; no longer IC6.28, IC6.6, Q1.3, X8.5
- net GND1: no longer IC6.18
- net MISO: now also J1.DAT0, U$9.MISO; no longer X8.2
- net MOSI: now also R8.2, U$9.MOSI; no longer X8.3
- net N$48: now also IC6.15; no longer Q1.1, Q1.2, Q1.5, Q1.6, X5.1
- net SCK: now also R7.2, U$9.SCK
- net SPI_CLK: no longer X8.1
- net VCC: no longer C17.1, C18.1, C19.1, C20.1, IC6.5, U1.2, U1.8
Routing:
- net +3V3: track 150.2 -> 29.7 mm, vias 1 -> 0
- net +5V: track 0.00 -> 57.5 mm
- net PW: track 49.0 -> 0.00 mm
- net VCC: track 25.9 -> 0.00 mm
- net SCL: track 14.7 -> 0.00 mm
- net GND1: track 209.3 -> 196.3 mm
- net N$48: track 12.0 -> 0.00 mm
- net +24V: track 64.0 -> 54.0 mm
- net N$25: track 8.14 -> 0.00 mm
- net MOSI: track 7.68 -> 0.00 mm
- net MISO: track 7.68 -> 0.00 mm
- net GND: track 63.3 -> 55.6 mm
- net N$20: track 5.21 -> 0.00 mm
- net N$23: track 4.96 -> 0.00 mm

Commit message: wip
Parts:
- removed D3: DIODE1N4007, MyLib:SMA-DIODE
- removed X9: MKDSN1,5/7-5,08, con-phoenix-508:MKDSN1,5/7-5,08
- added D14: BAV199, MyLib:SOT23
- added IC7: PCF8574T, micro-philips:SO16W
- added U$11, U$12, U$13, U$14: NSI45020AT1GSOD-123, MyLib:SOD123
- added U2: TRACO_TEL_5-1211, MyLib:TRACO_POWER_TL5
- added X2, X8: MKDSN1,5/4-5,08, con-phoenix-508:MKDSN1,5/4-5,08
- C1, C2, C4: device rcl:E3,5-8 -> rcl:153CLV-0605
- D1, D10, D12, D13, D2, D4, D5, D6, D7, D8, D9: value DIODE1N4007 -> BAV199; device MyLib:SMA-DIODE -> MyLib:SOT23
- moved C10 147.5 mm to (146.1, 33.7), turned to 270 degrees
- moved G1 137.7 mm to (14.8, 64.2)
- moved C9 114.0 mm to (91.3, 73.7), turned to 90 degrees
- moved C8 111.5 mm to (91.4, 44.7), turned to 180 degrees
- moved C5 103.9 mm to (-41.1, 75.6), turned to 270 degrees
- moved U$9 63.0 mm to (-6.16, 20.6), turned to 0 degrees
- moved D13 52.4 mm to (15.5, 12.7), turned to 180 degrees
- moved R10 39.6 mm to (119.4, 34.7)
- moved IC6 39.4 mm to (144.1, 50.9), turned to 90 degrees
- moved R12 38.0 mm to (-2.03, 77.0), turned to 90 degrees
- moved R6 35.6 mm to (-1.91, 65.1), turned to 90 degrees
- moved U$10 35.3 mm to (159.1, 45.7)
- moved X7 35.2 mm to (113.4, 35.9)
- moved R13 34.3 mm to (-8.70, 52.3), turned to 270 degrees
- moved JP4 33.5 mm to (-1.65, 52.3)
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Connections:
- net N$73 renamed I_CONTRAST
- net R/W renamed 485_R/W
- removed net ID0: IC6.9, U$10.21, U$10.7
- removed net ID1: IC6.10, U$10.22, U$10.8
- removed net ID2: IC6.11, U$10.23, U$10.9
- removed net ID3: IC6.12, U$10.10, U$10.24
- removed net N$52: IC4.5, JP1.9
- removed net N$61: IC6.14
- removed net PE: C13.2, C15.2, C16.2, D11.3, GDT1.1, GDT2.2, L2.2, U1.16, U1.20, X1.2
- removed net RS2: IC2.1
- removed net SPI_CLK: X6.1
- removed net VCC: IC2.4, IC2.6
- new net INT1: IC2.1, IC5.13
- new net I_D0: IC7.4, U$10.21, U$10.7
- new net I_D1: IC7.5, U$10.22, U$10.8
- new net I_D2: IC7.6, U$10.23, U$10.9
- new net I_D3: IC7.7, U$10.10, U$10.24
- new net I_D4: IC7.9, U$10.11, U$10.25
- new net I_D5: IC7.10, U$10.12, U$10.26
- new net I_D6: IC7.11, U$10.13, U$10.27
- new net I_D7: IC7.12, U$10.14, U$10.28
- new net N$62: U$11.C, X3.1
- new net N$63: U$12.C, X3.2
- new net N$65: U$13.C, X3.3
- new net N$67: U$14.C, X3.4
- net +24V: now also D1.2, D10.2, D12.2, D13.2, D14.2, D2.2, D4.2, D5.2, D6.2, D7.2, D8.2, D9.2, U2.+VIN@1, U2.+VIN@2
- net +3V3: no longer C10.1, C8.1, C9.1
- net +5V: now also C10.1, C8.1, C9.1, IC2.4, IC2.6, IC7.1, IC7.16, IC7.2, U2.+VOUT
- net E_SELECT: now also IC2.14
- net GND: now also IC7.3, IC7.8, U2.-VOUT
- net GND1: now also C13.2, C15.2, C16.2, D1.1, D10.1, D11.3, D12.1, D13.1, D14.1, D2.1, D4.1, D5.1, D6.1, D7.1, D8.1, D9.1, GDT1.1, GDT2.2, L2.2, U1.16, U1.20, U2.-VIN@1, U2.-VIN@2, X1.2; no longer D1.A, D10.A, D12.A, D13.A, D2.A, D3.A, D4.A, D5.A, D6.A, D7.A, D8.A, D9.A, X9.1
- net INT-S: no longer IC5.13
- net I_E: now also IC6.10; no longer IC6.7
- net I_RS: now also IC6.12; no longer IC6.5
- net I_RW: now also IC6.11; no longer IC6.6
- net N$10: now also D13.3, U$11.A; no longer D4.C, X3.1
- net N$11: now also D4.3, U$12.A; no longer D1.C, X3.2
- net N$12: now also D1.3, U$13.A; no longer D2.C, X3.3
- net N$13: now also D2.3, U$14.A; no longer D3.C, X3.4
- net N$16: now also D14.3; no longer D5.C
- net N$17: now also D5.3; no longer D6.C
- net N$21: now also X2.4; no longer X9.7
- net N$22: now also X2.3; no longer X9.6
- net N$24: now also D6.3; no longer D7.C
- net N$27: now also D7.3, OC4.1, U$5.C; no longer D12.C, OC11.1, U$3.C
- net N$28: now also X8.2
- net N$30: now also D8.3, OC5.1, U$6.C; no longer D8.C, OC4.1, U$5.C
- net N$32: now also D9.3, OC6.1, U$7.C; no longer D9.C, OC5.1, U$6.C
- net N$33: now also X2.1; no longer X9.4
- net N$34: now also D10.3, OC11.1, U$3.C; no longer D13.C, OC12.1, U$8.C
- net N$35: now also X2.2; no longer X9.5
- net N$36: now also D12.3, OC12.1, U$8.C; no longer D10.C, OC6.1, U$7.C
- net N$37: now also X8.4; no longer X9.3
- net N$38: now also X8.3; no longer X9.2
- net N$39: now also X8.1
- net N$48: now also IC4.5, JP1.6; no longer IC6.15
- net N$50: now also JP1.9; no longer JP1.6
- net SCK: now also X6.1
- net SCL: now also IC6.14, IC7.14
- net SDA: now also IC6.15, IC7.15
- net SD_SELECT: now also IC2.9
Routing:
- net +5V: track 57.5 -> 494.0 mm, vias 0 -> 12
- net GND: track 55.6 -> 351.3 mm
- net SCL: track 0.00 -> 207.9 mm, vias 0 -> 5
- net +24V: track 54.0 -> 258.8 mm, vias 0 -> 2
- net SDA: track 0.00 -> 190.3 mm, vias 0 -> 7
- net GND1: track 196.3 -> 58.9 mm
- net INT1: track 0.00 -> 97.2 mm, vias 0 -> 2
- net MISO: track 0.00 -> 90.0 mm, vias 0 -> 3
- net SCK: track 0.00 -> 89.4 mm, vias 0 -> 2
- net MOSI: track 0.00 -> 88.9 mm, vias 0 -> 2
- net I_D7: track 0.00 -> 73.0 mm, vias 0 -> 1
- net I_D6: track 0.00 -> 65.8 mm, vias 0 -> 1
- net I_D5: track 0.00 -> 64.7 mm, vias 0 -> 1
- net N$20: track 0.00 -> 60.4 mm, vias 0 -> 2
- net I_D3: track 0.00 -> 58.5 mm, vias 0 -> 1
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- added copper zone on layer 1, net GND
- added copper zone on layer 1, net GND1
Other:
- board size 168.4 x 86.7 mm -> 192.7 x 86.7 mm

Commit message: All routed.
Parts:
- flipped X2 to the bottom
- flipped X8 to the bottom
Connections:
- net N$21: now also X2.1; no longer X2.4
- net N$22: now also X2.2; no longer X2.3
- net N$28: now also X8.3; no longer X8.2
- net N$33: now also X2.4; no longer X2.1
- net N$35: now also X2.3; no longer X2.2
- net N$37: now also X8.1; no longer X8.4
- net N$38: now also X8.2; no longer X8.3
- net N$39: now also X8.4; no longer X8.1
Routing:
- net +5V: track 494.0 -> 507.3 mm
- net +3V3: track 54.3 -> 66.8 mm
- net N$21: track 13.6 -> 11.1 mm
- net N$39: track 10.6 -> 8.09 mm
- net N$33: track 10.6 -> 8.12 mm
- net N$37: track 14.2 -> 12.0 mm
- net N$38: track 7.82 -> 9.98 mm
Changed lines of the file:
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@@
 <element name="C10" library="rcl" package="C0805" value="0.1" x="146.1135" y="33.7185" rot="R270"/>
 <element name="U2" library="MyLib" package="TRACO_POWER_TL5" value="TRACO_TEL_5-1211" x="149.5425" y="23.3045" rot="R90"/>
-<element name="X2" library="con-phoenix-508" package="MKDSN1,5/4-5,08" value="MKDSN1,5/4-5,08" x="117.7925" y="1.8415"/>
-<element name="X8" library="con-phoenix-508" package="MKDSN1,5/4-5,08" value="MKDSN1,5/4-5,08" x="81.3435" y="1.905"/>
+<element name="X2" library="con-phoenix-508" package="MKDSN1,5/4-5,08" value="MKDSN1,5/4-5,08" x="117.7925" y="1.8415" rot="MR0"/>
+<element name="X8" library="con-phoenix-508" package="MKDSN1,5/4-5,08" value="MKDSN1,5/4-5,08" x="81.3435" y="1.905" rot="MR0"/>
 <element name="D14" library="MyLib" package="SOT23" value="BAV199" x="128.8415" y="12.7635" rot="R180"/>
 <element name="D5" library="MyLib" package="SOT23" value="BAV199" x="119.888" y="12.7635" rot="R180"/>
@@
 <wire x1="-6.493" y1="67.152" x2="-25.908" y2="67.152" width="0.4064" layer="1"/>
 <wire x1="-25.908" y1="46.6725" x2="-25.908" y2="67.152" width="0.4064" layer="1"/>
-<wire x1="-17.0485" y1="41.148" x2="-17.0485" y2="46.6725" width="0.4064" layer="1"/>
+<wire x1="-17.0485" y1="46.6725" x2="-17.0485" y2="41.148" width="0.4064" layer="1"/>
 <wire x1="-17.0485" y1="46.6725" x2="-25.908" y2="46.6725" width="0.4064" layer="1"/>
+<wire x1="-17.0485" y1="41.148" x2="-17.0485" y2="38.3235" width="0.4064" layer="1"/>
+<wire x1="-17.0485" y1="38.3235" x2="-19.05" y2="36.322" width="0.4064" layer="1"/>
+<wire x1="-19.05" y1="36.322" x2="-19.05" y2="34.859" width="0.4064" layer="1"/>
+<wire x1="-19.05" y1="34.859" x2="-18.989" y2="34.798" width="0.4064" layer="1"/>
+<wire x1="-18.989" y1="34.798" x2="-18.989" y2="30.2745" width="0.4064" layer="1"/>
+<wire x1="-18.989" y1="30.2745" x2="-19.558" y2="29.7055" width="0.4064" layer="1"/>
 <wire x1="-17.0485" y1="46.6725" x2="-8.6995" y2="51.374" width="0" layer="19" extent="1-1"/>
-<wire x1="-18.989" y1="34.798" x2="-17.0485" y2="41.148" width="0" layer="19" extent="1-1"/>
-<wire x1="-19.558" y1="29.7055" x2="-18.989" y2="34.798" width="0" layer="19" extent="1-1"/>
 <wire x1="-19.558" y1="23.5075" x2="-19.558" y2="29.7055" width="0" layer="19" extent="1-1"/>
 <wire x1="-41.148" y1="76.5785" x2="-25.908" y2="67.152" width="0" layer="19" extent="1-1"/>
@@
 <wire x1="150.9395" y1="48.9585" x2="150.9395" y2="46.4185" width="0.4064" layer="1"/>
 <wire x1="150.9395" y1="46.4185" x2="148.6815" y2="46.4185" width="0.4064" layer="1"/>
-<wire x1="163.3855" y1="74.422" x2="163.2585" y2="74.422" width="0.8128" layer="1"/>
-<wire x1="163.2585" y1="74.422" x2="163.2585" y2="74.295" width="0.8128" layer="1"/>
+<wire x1="163.3855" y1="74.422" x2="163.2585" y2="74.422" width="0" layer="19" extent="1-16"/>
+<wire x1="163.2585" y1="74.422" x2="163.2585" y2="74.295" width="0" layer="19" extent="1-16"/>
 <wire x1="128.9685" y1="31.242" x2="128.9685" y2="48.895" width="0.4064" layer="1"/>
 <wire x1="63.4085" y1="49.53" x2="61.4045" y2="49.53" width="0.4064" layer="1"/>
@@
 <signal name="N$22">
 <contactref element="U$2" pad="A"/>
-<contactref element="X2" pad="3"/>
-<wire x1="123.693" y1="8.255" x2="123.693" y2="6.5355" width="0.4064" layer="1"/>
-<wire x1="123.693" y1="6.5355" x2="120.3325" y2="3.175" width="0.4064" layer="1"/>
-<wire x1="120.3325" y1="3.175" x2="120.3325" y2="1.8876" width="0.4064" layer="1"/>
-<wire x1="120.3325" y1="1.8876" x2="120.3114" y2="1.8665" width="0.4064" layer="1"/>
+<contactref element="X2" pad="2"/>
+<wire x1="120.3536" y1="1.8665" x2="123.693" y2="5.2059" width="0.4064" layer="1"/>
+<wire x1="123.693" y1="5.2059" x2="123.693" y2="8.255" width="0.4064" layer="1"/>
 </signal>
 <signal name="GND1">
@@
 <signal name="N$35">
 <contactref element="U$4" pad="A"/>
-<contactref element="X2" pad="2"/>
-<wire x1="115.1205" y1="8.255" x2="115.1205" y2="1.8665" width="0.4064" layer="1"/>
-<wire x1="115.1205" y1="1.8665" x2="115.2314" y2="1.8665" width="0.4064" layer="1"/>
+<contactref element="X2" pad="3"/>
+<wire x1="115.2736" y1="1.8665" x2="115.1205" y2="2.0196" width="0.4064" layer="1"/>
+<wire x1="115.1205" y1="2.0196" x2="115.1205" y2="8.255" width="0.4064" layer="1"/>
 </signal>
 <signal name="N$37">
 <contactref element="U$6" pad="A"/>
-<contactref element="X8" pad="4"/>
-<wire x1="96.896" y1="8.1915" x2="96.896" y2="1.93" width="0.4064" layer="1"/>
-<wire x1="96.896" y1="1.93" x2="88.9424" y2="1.93" width="0.4064" layer="1"/>
+<contactref element="X8" pad="1"/>
+<wire x1="88.9846" y1="1.93" x2="92.6426" y2="5.588" width="0.4064" layer="1"/>
+<wire x1="92.6426" y1="5.588" x2="96.901" y2="5.588" width="0.4064" layer="1"/>
+<wire x1="96.901" y1="5.588" x2="96.896" y2="5.593" width="0.4064" layer="1"/>
+<wire x1="96.896" y1="5.593" x2="96.896" y2="8.1915" width="0.4064" layer="1"/>
 </signal>
 <signal name="N$33">
 <contactref element="U$5" pad="A"/>
-<contactref element="X2" pad="1"/>
-<wire x1="105.8495" y1="8.1915" x2="105.8495" y2="1.8665" width="0.4064" layer="1"/>
-<wire x1="105.8495" y1="1.8665" x2="110.1514" y2="1.8665" width="0.4064" layer="1"/>
+<contactref element="X2" pad="4"/>
+<wire x1="110.1936" y1="1.8665" x2="105.8495" y2="6.2106" width="0.4064" layer="1"/>
+<wire x1="105.8495" y1="6.2106" x2="105.8495" y2="8.1915" width="0.4064" layer="1"/>
 </signal>
 <signal name="N$38">
 <contactref element="U$7" pad="A"/>
-<contactref element="X8" pad="3"/>
-<wire x1="87.6885" y1="8.128" x2="87.6885" y2="7.107" width="0.4064" layer="1"/>
-<wire x1="87.6885" y1="7.107" x2="83.82" y2="3.2385" width="0.4064" layer="1"/>
-<wire x1="83.82" y1="3.2385" x2="83.82" y2="1.9724" width="0.4064" layer="1"/>
-<wire x1="83.82" y1="1.9724" x2="83.8624" y2="1.93" width="0.4064" layer="1"/>
+<contactref element="X8" pad="2"/>
+<wire x1="87.6885" y1="8.128" x2="87.6885" y2="5.0165" width="0.4064" layer="1"/>
+<wire x1="87.6885" y1="5.0165" x2="84.0105" y2="5.0165" width="0.4064" layer="1"/>
+<wire x1="84.0105" y1="5.0165" x2="84.0105" y2="1.93" width="0.4064" layer="1"/>
+<wire x1="84.0105" y1="1.93" x2="83.9046" y2="1.93" width="0.4064" layer="1"/>
 </signal>
 <signal name="INT0">
@@
 <wire x1="-22.2885" y1="62.0395" x2="-22.352" y2="62.103" width="0.8128" layer="16"/>
 <via x="-22.352" y="62.103" extent="1-16" drill="0.6"/>
-<wire x1="-17.112" y1="11.684" x2="-13.0175" y2="11.684" width="0.4064" layer="1"/>
+<wire x1="-13.0175" y1="11.684" x2="-17.112" y2="11.684" width="0.4064" layer="1"/>
 <wire x1="-13.0175" y1="41.3385" x2="-13.0175" y2="11.684" width="0.4064" layer="1"/>
 <wire x1="-13.0175" y1="41.3385" x2="-13.0175" y2="52.832" width="0.4064" layer="1"/>
@@
 <wire x1="148.6535" y1="74.422" x2="148.6535" y2="78.736" width="0.8128" layer="1"/>
 <wire x1="148.6535" y1="78.736" x2="148.6575" y2="78.74" width="0.8128" layer="1"/>
+<wire x1="-17.247" y1="18.9865" x2="-17.247" y2="23.5075" width="0.4064" layer="1"/>
+<wire x1="-17.247" y1="18.9865" x2="-18.608" y2="18.9865" width="0.4064" layer="1"/>
+<wire x1="-17.112" y1="11.684" x2="-17.112" y2="18.9865" width="0.4064" layer="1"/>
+<wire x1="-17.112" y1="18.9865" x2="-17.247" y2="18.9865" width="0.4064" layer="1"/>
 <wire x1="91.313" y1="72.7735" x2="99.441" y2="92.456" width="0" layer="19" extent="1-1"/>
 <wire x1="94.615" y1="61.9125" x2="91.313" y2="72.7735" width="0" layer="19" extent="1-1"/>
-<wire x1="-18.608" y1="18.9865" x2="-17.112" y2="11.684" width="0" layer="19" extent="1-1"/>
-<wire x1="-17.247" y1="23.5075" x2="-18.608" y2="18.9865" width="0" layer="19" extent="1-1"/>
 </signal>
 <signal name="SCK">
@@
 <signal name="N$28">
 <contactref element="U$3" pad="A"/>
-<contactref element="X8" pad="2"/>
+<contactref element="X8" pad="3"/>
 <wire x1="78.7985" y1="8.128" x2="78.7985" y2="1.93" width="0.4064" layer="1"/>
-<wire x1="78.7985" y1="1.93" x2="78.7824" y2="1.93" width="0.4064" layer="1"/>
+<wire x1="78.7985" y1="1.93" x2="78.8246" y2="1.93" width="0.4064" layer="1"/>
 </signal>
 <signal name="N$39">
 <contactref element="U$8" pad="A"/>
-<contactref element="X8" pad="1"/>
-<wire x1="69.337" y1="8.1915" x2="69.337" y2="1.93" width="0.4064" layer="1"/>
-<wire x1="69.337" y1="1.93" x2="73.7024" y2="1.93" width="0.4064" layer="1"/>
+<contactref element="X8" pad="4"/>
+<wire x1="73.7446" y1="1.93" x2="69.337" y2="6.3376" width="0.4064" layer="1"/>
+<wire x1="69.337" y1="6.3376" x2="69.337" y2="8.1915" width="0.4064" layer="1"/>
 </signal>
 <signal name="N$41">
@@
 <signal name="N$21">
 <contactref element="U$1" pad="A"/>
-<contactref element="X2" pad="4"/>
-<wire x1="132.6465" y1="8.255" x2="132.6465" y2="1.8665" width="0.4064" layer="1"/>
-<wire x1="132.6465" y1="1.8665" x2="125.3914" y2="1.8665" width="0.4064" layer="1"/>
+<contactref element="X2" pad="1"/>
+<wire x1="125.4336" y1="1.8665" x2="129.7266" y2="6.1595" width="0.4064" layer="1"/>
+<wire x1="129.7266" y1="6.1595" x2="132.6515" y2="6.1595" width="0.4064" layer="1"/>
+<wire x1="132.6515" y1="6.1595" x2="132.6465" y2="6.1645" width="0.4064" layer="1"/>
+<wire x1="132.6465" y1="6.1645" x2="132.6465" y2="8.255" width="0.4064" layer="1"/>
 </signal>
 <signal name="N$16">

Commit message: wip
Parts:
- added C21, C22: 0.1, rcl:C0805
- moved X4 78.6 mm to (128.9, 77.6), turned to 0 degrees
- moved X5 66.7 mm to (131.4, 35.2), turned to 270 degrees
- moved C6 65.9 mm to (128.9, 71.0), turned to 180 degrees
- moved C9 59.5 mm to (32.1, 67.8), turned to 0 degrees
- moved C4 54.6 mm to (129.1, 65.0), turned to 0 degrees
- moved IC7 54.3 mm to (73.2, 62.0)
- moved IC6 45.2 mm to (98.9, 51.8)
- moved G1 44.0 mm to (58.4, 69.8), turned to 180 degrees
- moved U$10 43.1 mm to (116.0, 46.1)
- moved U2 38.6 mm to (129.3, 56.2), turned to 270 degrees
- moved R9 31.9 mm to (-19.1, 52.3)
- moved C7 29.3 mm to (-20.8, 5.52), turned to 0 degrees
- moved C1 28.5 mm to (-19.0, 12.7), turned to 180 degrees
- moved R12 28.3 mm to (-15.8, 52.3)
- moved C2 26.1 mm to (-16.6, 37.6), turned to 180 degrees
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Connections:
- net +5V: now also C21.1, C22.1
- net 485_R/W: now also IC2.2; no longer IC2.12
- net GND: now also C21.2, C22.2
- net SD_SELECT: now also IC2.13; no longer IC2.9
Routing:
- net GND: track 351.0 -> 216.5 mm
- net +5V: track 507.3 -> 433.5 mm
- net SCL: track 207.9 -> 152.2 mm, vias 5 -> 7
- net E_SELECT: track 0.00 -> 51.7 mm, vias 0 -> 1
- net SDA: track 190.3 -> 141.1 mm, vias 7 -> 6
- net +24V: track 258.8 -> 307.2 mm
- net N$20: track 60.4 -> 18.2 mm, vias 2 -> 0
- net +3V3: track 66.8 -> 96.1 mm, vias 0 -> 2
- net SD_SELECT: track 38.0 -> 60.0 mm
- net N$6: track 42.2 -> 21.6 mm
- net N$9: track 50.4 -> 32.5 mm
- net N$29: track 3.23 -> 20.4 mm
- net N$8: track 43.8 -> 27.8 mm
- net N$7: track 39.0 -> 24.3 mm
- net N$43: track 0.00 -> 13.9 mm
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Other:
- board size 192.7 x 86.7 mm -> 173.2 x 86.7 mm

Commit message: Ready to gerber
Parts:
- added C23, C24, C25, C26: 0.1, rcl:C0805
- added IC8: DS1813-SMD, MyLib:SOT-23
- added JP2: (no value), pinhead:1X03
- added JP3: (no value), pinhead:1X04
- moved C7 8.34 mm to (-22.0, 13.8), turned to 270 degrees
- moved Q5 7.06 mm to (42.5, 75.0)
- moved C1 2.21 mm to (-16.9, 12.0), turned to 90 degrees
- moved C17 1.40 mm to (56.2, 48.6)
- moved C3 1.31 mm to (-15.7, 30.8)
- moved C20 1.14 mm to (45.7, 51.8)
- moved C19 1.08 mm to (45.7, 48.6)
- moved C18 1.08 mm to (56.2, 51.8)
- moved C9 0.99 mm to (33.0, 67.3), turned to 270 degrees
- moved C2 0.06 mm to (-16.6, 37.6)
Connections:
- removed net AVCC: IC2.18
- new net N$61: C23.1, IC2.20
- new net N$64: IC2.10, JP3.3
- new net N$66: IC2.9, JP3.4
- net +24V: now also C24.1, C25.1, C26.1
- net +5V: now also IC2.18, IC8.2, JP2.2, JP3.1
- net E_RESET: now also IC2.13
- net GND: now also C23.2, IC8.3, JP2.1, JP3.2
- net GND1: now also C24.2, C25.2, C26.2
- net I_CONTRAST: now also JP2.3
- net I_E: now also IC6.9; no longer IC6.10
- net I_RS: now also IC6.11; no longer IC6.12
- net I_RW: now also IC6.10; no longer IC6.11
- net RESET: now also IC8.1
- net SD_DETECT: now also IC2.11
- net SD_SELECT: now also IC2.12; no longer IC2.13
- net SPI0: now also IC2.19
Routing:
- net E_RESET: track 0.00 -> 63.9 mm, vias 0 -> 1
- net SD_DETECT: track 4.05 -> 52.3 mm, vias 0 -> 2
- net SPI0: track 0.00 -> 30.5 mm
- net +5V: track 433.5 -> 462.6 mm, vias 12 -> 13
- net GND: track 216.5 -> 191.8 mm
- net +24V: track 307.2 -> 321.1 mm
- net N$64: track 0.00 -> 13.2 mm
- net N$66: track 0.00 -> 11.8 mm
- net N$61: track 0.00 -> 9.06 mm
- net MOSI: track 89.8 -> 81.9 mm, vias 5 -> 4
- net RESET: track 42.5 -> 49.0 mm, vias 1 -> 2
- net +3V3: track 96.1 -> 89.8 mm
- net N$25: track 5.29 -> 11.4 mm
- net N$23: track 5.29 -> 10.6 mm
- net SD_SELECT: track 60.0 -> 55.4 mm
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