File: sortirovka.sch (EAGLE design)
At the start: 19 parts, among them U1 MAX3485CSA, X1 PI3-CON, X2 MKDSN1,5/2-5,08, X3 MKDSN1,5/4-5,08, X4 MKDSN1,5/2-5,08

Commit message: rev1
Parts:
- added D5, D6: BAV199, diode:BAV199
- added G1: CR2032H, MyLib:CR2032H
- added IC1: DS1307Z, MyLib:DS1307Z
- added OC1, OC2: (no value), MyLib:SFH6106
- added Q5: (no value), MyLib:MA306
- added R10, R11: 3k3, rcl:R-EU_R0805
- added R5, R6: 10k, rcl:R-EU_R0805
- added R7: 0, rcl:R-EU_R0805
- added R8, R9: 100, rcl:R-EU_R0805
- added U$1, U$2: NSI45020AT1GSOD-123, MyLib:NSI45020AT1GSOD-123
- added U$3: NUP2105LSOT23-R, MyLib:NUP2105LSOT23-R
- added X5: MKDSN1,5/3-5,08, con-phoenix-508:MKDSN1,5/3-5,08
- added X6, X8: 22-23-2051, con-molex:22-23-2051
- added X7: 22-23-2041, con-molex:22-23-2041
- R1, R2, R3, R4: value (none) -> 10k
Connections:
- new net +5V: IC1.VCC
- new net MISO: X1.GPIO09, X6-4.S, X8-4.S
- new net MOSI: X1.GPIO10, X6-5.S, X8-5.S
- new net N$14: R7.1, X1.3.3V@1, X1.3.3V@2
- new net N$15: OC2.EMIT, R6.2, X1.GPIO06
- new net N$16: OC1.A, U$1.C
- new net N$17: OC2.A, U$2.C
- new net N$18: OC1.EMIT, R5.2, X1.GPIO05
- new net N$19: D5.AC, R8.1, U$1.A
- new net N$20: G1.+, IC1.VBAT
- new net N$21: R8.2, X5-3.KL
- new net N$22: R9.2, X5-1.KL
- new net N$23: IC1.X1, Q5.1
- new net N$24: D6.AC, R9.1, U$2.A
- new net N$25: IC1.X2, Q5.2
- new net N$26: IC1.SCL, R10.1, X1.GPIO03, X7-2.S
- new net N$27: IC1.SDA, R11.1, X1.GPIO02, X7-1.S
- new net SPI0: X1.GPIO08, X6-2.S
- new net SPI1: X1.GPIO07, X8-2.S
- new net SPI_CLK: X1.GPIO11, X6-3.S, X8-3.S
- net +24V: now also D5.C, D6.C
- net +3V3: now also OC1.COL, OC2.COL, R10.2, R11.2, R7.2, X7-3.S; no longer X1.3.3V@1, X1.3.3V@2
- net GND: now also D5.A, D6.A, G1.-, IC1.GND, OC1.C, OC2.C, R5.1, R6.1, U$3.P$3, X1.GND@2, X1.GND@5, X5-2.KL, X6-1.S, X7-4.S, X8-1.S
- net N$4: now also U$3.P$2, U1.A; no longer U1.B
- net N$5: now also U$3.P$1, U1.B; no longer U1.A
Other:
- note added: "(PCF85263A)"
- moved on the sheet: C1, C2, D1, D2, D3, D4, Q1, Q2, Q3, Q4, R1, R2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

Commit message: rev2 5-input 4-output
Parts:
- removed C1, C2: (no value), rcl:C-EUC0805K
- removed D5, D6: BAV199, diode:BAV199
- removed X5: MKDSN1,5/3-5,08, con-phoenix-508:MKDSN1,5/3-5,08
- added JP1: (no value), pinhead:PINHD-1X1
- added OC3, OC4, OC5: (no value), MyLib:SFH6106
- added R12: 10k, rcl:R-EU_R0805
- added U$4, U$5, U$6: NSI45020AT1GSOD-123, MyLib:NSI45020AT1GSOD-123
- added X9: MKDSN1,5/7-5,08, con-phoenix-508:MKDSN1,5/7-5,08
- R8, R9: value 100 -> 10k
Connections:
- new net GND1: D1.A, D2.A, D3.A, D4.A, OC1.C, OC2.C, OC3.C, OC4.C, OC5.C, X4-2.KL, X9-1.KL
- new net N$28: JP1.1, X1.+5V@1, X1.+5V@2
- new net N$29: OC4.EMIT, R9.2, X1.GPIO19
- new net N$30: OC4.A, U$5.C
- new net N$31: OC5.EMIT, R12.2, X1.GPIO26
- new net N$32: OC5.A, U$6.C
- new net N$33: U$5.A, X9-4.KL
- new net N$35: U$4.A, X9-5.KL
- new net N$37: U$6.A, X9-3.KL
- net +24V: no longer C1.1, C2.1, D5.C, D6.C
- net +3V3: now also OC3.COL, OC4.COL, OC5.COL, X7-1.S; no longer X7-3.S
- net GND: now also R12.1, R8.1, R9.1; no longer C1.2, C2.2, D1.A, D2.A, D3.A, D4.A, D5.A, D6.A, OC1.C, OC2.C, X4-2.KL, X5-2.KL
- net N$11: now also D1.C; no longer D3.C
- net N$13: now also D3.C; no longer D1.C
- net N$19: now also OC3.EMIT, R8.2, X1.GPIO13; no longer D5.AC, R8.1, U$1.A
- net N$21: now also U$1.A, X9-7.KL; no longer R8.2, X5-3.KL
- net N$22: now also U$2.A, X9-6.KL; no longer R9.2, X5-1.KL
- net N$24: now also OC3.A, U$4.C; no longer D6.AC, R9.1, U$2.A
- net N$26: now also X7-3.S; no longer X7-2.S
- net N$27: now also X7-2.S; no longer X7-1.S
Other:
- moved on the sheet: D1, D2, D3, D4, R8, R9, X4-1, X4-2

Commit message: rev1.0 to produce
Parts:
- removed JP1: (no value), pinhead:PINHD-1X1
- removed Q1, Q2, Q3, Q4: (no value), MyLib:MOSFET-NWIDE
- removed X2: MKDSN1,5/2-5,08, con-phoenix-508:MKDSN1,5/2-5,08
- added C1, C2, C4: (no value), rcl:CPOL-EUSANYO_C
- added C10, C3, C5, C6, C7, C8, C9: 0.1, rcl:C-EUC0805
- added D10, D5, D6, D7, D8, D9: DIODE1N4007, MyLib:DIODE1N4007
- added IC3: LM1117IMPX-3.3, lm1117:LM1117IMPX-3.3
- added JP2: (no value), pinhead:PINHD-1X1
- added OC10, OC6, OC7, OC8, OC9: (no value), MyLib:SFH6106
- added R13: 10k, rcl:R-EU_R0805
- added R14: 0, rcl:R-EU_R0805
- added R15: 120, rcl:R-EU_0204/7
- added R16, R17: 47, rcl:R-EU_0204/7
- added R18, R19, R20: 560, rcl:R-EU_0204/7
- added U$7: NSI45020AT1GSOD-123, MyLib:NSI45020AT1GSOD-123
- added X10: MKDSN1,5/3-5,08, con-phoenix-508:MKDSN1,5/3-5,08
- added X5: 22-23-2021, con-molex:22-23-2021
- R1, R2, R3, R4: value 10k -> 200
Connections:
- removed net +5V: IC1.VCC
- removed net N$31: OC5.EMIT, R12.2, X1.GPIO26
- new net N$34: OC6.EMIT, R13.2, X1.GPIO26
- new net N$36: D10.C, OC6.A, U$7.C
- new net N$38: U$7.A, X9-2.KL
- new net N$39: OC5.EMIT, R12.2, X1.GPIO19
- new net N$40: OC4.EMIT, R9.2, X1.GPIO13
- new net N$41: OC3.EMIT, R8.2, X1.GPIO06
- new net N$42: OC2.EMIT, R6.2, X1.GPIO05
- new net N$43: JP2.1, OC1.EMIT, R5.2, X1.GPIO04
- new net N$45: R15.2, R16.1, X10-2.KL
- new net N$46: R15.1, R17.1, X10-1.KL
- new net N$47: R17.2, R19.1, U$3.P$2, U1.A
- new net PW: C2.+, C3.1, IC3.IN, R14.2, X5-1.S
- net +24V: now also C4.+, C6.1, OC10.COL, OC7.COL, OC8.COL, OC9.COL; no longer Q1.D, Q2.D, Q3.D, Q4.D
- net +3V3: now also C1.+, C10.1, C5.1, C7.1, C8.1, C9.1, IC1.VCC, IC3.OUT, IC3.OUT1, OC6.COL, R19.2
- net GND: now also C1.-, C10.2, C2.-, C3.2, C5.2, C7.2, C8.2, C9.2, IC3.GND, OC10.C, OC7.C, OC8.C, OC9.C, R13.1, R18.1, R20.2, X5-2.S, X6-5.S, X8-5.S; no longer R1.1, R2.1, R3.1, R4.1, X6-1.S, X8-1.S
- net GND1: now also C4.-, C6.2, D10.A, D5.A, D6.A, D7.A, D8.A, D9.A, OC6.C
- net MISO: now also X6-2.S, X8-2.S; no longer X6-4.S, X8-4.S
- net MOSI: now also X6-3.S, X8-3.S; no longer X6-5.S, X8-5.S
- net N$10: now also OC10.EMIT; no longer Q4.S
- net N$11: now also OC9.EMIT; no longer Q3.S
- net N$12: now also OC8.EMIT; no longer Q2.S
- net N$13: now also OC7.EMIT; no longer Q1.S
- net N$15: now also OC7.A, R1.1; no longer OC2.EMIT, R6.2, X1.GPIO06
- net N$16: now also D5.C
- net N$17: now also D6.C
- net N$18: now also OC8.A, R2.1; no longer OC1.EMIT, R5.2, X1.GPIO05
- net N$19: now also OC9.A, R3.1; no longer OC3.EMIT, R8.2, X1.GPIO13
- net N$24: now also D7.C
- net N$28: now also R14.1; no longer JP1.1
- net N$29: now also OC10.A, R4.1; no longer OC4.EMIT, R9.2, X1.GPIO19
- net N$30: now also D8.C
- net N$32: now also D9.C
- net N$4: now also R16.2, R18.2, U$3.P$1, U1.B; no longer U$3.P$2, U1.A, X2-1.KL
- net N$5: now also R20.1, X10-3.KL; no longer U$3.P$1, U1.B, X2-2.KL
- net N$6: no longer Q1.G
- net N$7: no longer Q2.G
- net N$8: no longer Q3.G
- net N$9: no longer Q4.G
- net SPI0: now also X6-4.S; no longer X6-2.S
- net SPI1: now also X8-4.S; no longer X8-2.S
- net SPI_CLK: now also X6-1.S, X8-1.S; no longer X6-3.S, X8-3.S
Other:
- note added: "A(+)"
- note added: "B(-)"
- moved on the sheet: D1, D2, D3, D4, OC1, OC2, OC3, OC4, OC5, R1, R12, R2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

Commit message: some changes in packages
Parts:
- C1, C2, C4: device rcl:CPOL-EUSANYO_C -> rcl:CPOL-EUE3.5-8
- R15, R16, R17, R18, R19, R20: device rcl:R-EU_0204/7 -> rcl:R-EU_0207/10
Changed lines of the file:
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@@
 <grid distance="0.1" unitdist="inch" unit="inch" style="lines" multiple="1" display="no" altdistance="0.01" altunitdist="inch" altunit="inch"/>
 <layers>
-<layer number="1" name="Top" color="4" fill="1" visible="no" active="no"/>
-<layer number="2" name="Route2" color="1" fill="3" visible="no" active="no"/>
-<layer number="3" name="Route3" color="4" fill="3" visible="no" active="no"/>
-<layer number="4" name="Route4" color="1" fill="4" visible="no" active="no"/>
-<layer number="5" name="Route5" color="4" fill="4" visible="no" active="no"/>
-<layer number="6" name="Route6" color="1" fill="8" visible="no" active="no"/>
-<layer number="7" name="Route7" color="4" fill="8" visible="no" active="no"/>
-<layer number="8" name="Route8" color="1" fill="2" visible="no" active="no"/>
-<layer number="9" name="Route9" color="4" fill="2" visible="no" active="no"/>
-<layer number="10" name="Route10" color="1" fill="7" visible="no" active="no"/>
-<layer number="11" name="Route11" color="4" fill="7" visible="no" active="no"/>
-<layer number="12" name="Route12" color="1" fill="5" visible="no" active="no"/>
-<layer number="13" name="Route13" color="4" fill="5" visible="no" active="no"/>
-<layer number="14" name="Route14" color="1" fill="6" visible="no" active="no"/>
-<layer number="15" name="Route15" color="4" fill="6" visible="no" active="no"/>
-<layer number="16" name="Bottom" color="1" fill="1" visible="no" active="no"/>
-<layer number="17" name="Pads" color="2" fill="1" visible="no" active="no"/>
-<layer number="18" name="Vias" color="2" fill="1" visible="no" active="no"/>
-<layer number="19" name="Unrouted" color="6" fill="1" visible="no" active="no"/>
-<layer number="20" name="Dimension" color="15" fill="1" visible="no" active="no"/>
-<layer number="21" name="tPlace" color="7" fill="1" visible="no" active="no"/>
-<layer number="22" name="bPlace" color="7" fill="1" visible="no" active="no"/>
-<layer number="23" name="tOrigins" color="15" fill="1" visible="no" active="no"/>
-<layer number="24" name="bOrigins" color="15" fill="1" visible="no" active="no"/>
-<layer number="25" name="tNames" color="7" fill="1" visible="no" active="no"/>
-<layer number="26" name="bNames" color="7" fill="1" visible="no" active="no"/>
-<layer number="27" name="tValues" color="7" fill="1" visible="no" active="no"/>
-<layer number="28" name="bValues" color="7" fill="1" visible="no" active="no"/>
+<layer number="1" name="Top" color="4" fill="1" visible="yes" active="no"/>
+<layer number="2" name="Route2" color="1" fill="3" visible="yes" active="no"/>
+<layer number="3" name="Route3" color="4" fill="3" visible="yes" active="no"/>
+<layer number="4" name="Route4" color="1" fill="4" visible="yes" active="no"/>
+<layer number="5" name="Route5" color="4" fill="4" visible="yes" active="no"/>
+<layer number="6" name="Route6" color="1" fill="8" visible="yes" active="no"/>
+<layer number="7" name="Route7" color="4" fill="8" visible="yes" active="no"/>
+<layer number="8" name="Route8" color="1" fill="2" visible="yes" active="no"/>
+<layer number="9" name="Route9" color="4" fill="2" visible="yes" active="no"/>
+<layer number="10" name="Route10" color="1" fill="7" visible="yes" active="no"/>
+<layer number="11" name="Route11" color="4" fill="7" visible="yes" active="no"/>
+<layer number="12" name="Route12" color="1" fill="5" visible="yes" active="no"/>
+<layer number="13" name="Route13" color="4" fill="5" visible="yes" active="no"/>
+<layer number="14" name="Route14" color="1" fill="6" visible="yes" active="no"/>
+<layer number="15" name="Route15" color="4" fill="6" visible="yes" active="no"/>
+<layer number="16" name="Bottom" color="1" fill="1" visible="yes" active="no"/>
+<layer number="17" name="Pads" color="2" fill="1" visible="yes" active="no"/>
+<layer number="18" name="Vias" color="2" fill="1" visible="yes" active="no"/>
+<layer number="19" name="Unrouted" color="6" fill="1" visible="yes" active="no"/>
+<layer number="20" name="Dimension" color="15" fill="1" visible="yes" active="no"/>
+<layer number="21" name="tPlace" color="7" fill="1" visible="yes" active="no"/>
+<layer number="22" name="bPlace" color="7" fill="1" visible="yes" active="no"/>
+<layer number="23" name="tOrigins" color="15" fill="1" visible="yes" active="no"/>
+<layer number="24" name="bOrigins" color="15" fill="1" visible="yes" active="no"/>
+<layer number="25" name="tNames" color="7" fill="1" visible="yes" active="no"/>
+<layer number="26" name="bNames" color="7" fill="1" visible="yes" active="no"/>
+<layer number="27" name="tValues" color="7" fill="1" visible="yes" active="no"/>
+<layer number="28" name="bValues" color="7" fill="1" visible="yes" active="no"/>
 <layer number="29" name="tStop" color="7" fill="3" visible="no" active="no"/>
 <layer number="30" name="bStop" color="7" fill="6" visible="no" active="no"/>
@@
 <layer number="35" name="tGlue" color="7" fill="4" visible="no" active="no"/>
 <layer number="36" name="bGlue" color="7" fill="5" visible="no" active="no"/>
-<layer number="37" name="tTest" color="7" fill="1" visible="no" active="no"/>
-<layer number="38" name="bTest" color="7" fill="1" visible="no" active="no"/>
+<layer number="37" name="tTest" color="7" fill="1" visible="yes" active="no"/>
+<layer number="38" name="bTest" color="7" fill="1" visible="yes" active="no"/>
 <layer number="39" name="tKeepout" color="4" fill="11" visible="no" active="no"/>
 <layer number="40" name="bKeepout" color="1" fill="11" visible="no" active="no"/>
@@
 <layer number="44" name="Drills" color="7" fill="1" visible="no" active="no"/>
 <layer number="45" name="Holes" color="7" fill="1" visible="no" active="no"/>
-<layer number="46" name="Milling" color="3" fill="1" visible="no" active="no"/>
-<layer number="47" name="Measures" color="7" fill="1" visible="no" active="no"/>
-<layer number="48" name="Document" color="7" fill="1" visible="no" active="no"/>
-<layer number="49" name="Reference" color="7" fill="1" visible="no" active="no"/>
-<layer number="50" name="dxf" color="7" fill="1" visible="no" active="no"/>
-<layer number="51" name="tDocu" color="7" fill="1" visible="no" active="no"/>
-<layer number="52" name="bDocu" color="7" fill="1" visible="no" active="no"/>
-<layer number="53" name="tGND_GNDA" color="7" fill="9" visible="no" active="no"/>
-<layer number="54" name="bGND_GNDA" color="1" fill="9" visible="no" active="no"/>
-<layer number="56" name="wert" color="7" fill="1" visible="no" active="no"/>
-<layer number="57" name="tCAD" color="7" fill="1" visible="no" active="no"/>
-<layer number="59" name="tCarbon" color="7" fill="1" visible="no" active="no"/>
-<layer number="60" name="bCarbon" color="7" fill="1" visible="no" active="no"/>
+<layer number="46" name="Milling" color="3" fill="1" visible="yes" active="no"/>
+<layer number="47" name="Measures" color="7" fill="1" visible="yes" active="no"/>
+<layer number="48" name="Document" color="7" fill="1" visible="yes" active="no"/>
+<layer number="49" name="Reference" color="7" fill="1" visible="yes" active="no"/>
+<layer number="50" name="dxf" color="7" fill="1" visible="yes" active="no"/>
+<layer number="51" name="tDocu" color="7" fill="1" visible="yes" active="no"/>
+<layer number="52" name="bDocu" color="7" fill="1" visible="yes" active="no"/>
+<layer number="53" name="tGND_GNDA" color="7" fill="9" visible="yes" active="no"/>
+<layer number="54" name="bGND_GNDA" color="1" fill="9" visible="yes" active="no"/>
+<layer number="56" name="wert" color="7" fill="1" visible="yes" active="no"/>
+<layer number="57" name="tCAD" color="7" fill="1" visible="yes" active="no"/>
+<layer number="59" name="tCarbon" color="7" fill="1" visible="yes" active="no"/>
+<layer number="60" name="bCarbon" color="7" fill="1" visible="yes" active="no"/>
 <layer number="90" name="Modules" color="5" fill="1" visible="yes" active="yes"/>
 <layer number="91" name="Nets" color="2" fill="1" visible="yes" active="yes"/>
@@
 <part name="R14" library="rcl" deviceset="R-EU_" device="R0805" value="0"/>
 <part name="X10" library="con-phoenix-508" deviceset="MKDSN1,5/3-5,08" device=""/>
-<part name="C1" library="rcl" deviceset="CPOL-EU" device="SANYO_C"/>
-<part name="C2" library="rcl" deviceset="CPOL-EU" device="SANYO_C"/>
+<part name="C1" library="rcl" deviceset="CPOL-EU" device="E3.5-8"/>
+<part name="C2" library="rcl" deviceset="CPOL-EU" device="E3.5-8"/>
 <part name="C3" library="rcl" deviceset="C-EU" device="C0805" value="0.1"/>
-<part name="R15" library="rcl" deviceset="R-EU_" device="0204/7" value="120"/>
-<part name="R16" library="rcl" deviceset="R-EU_" device="0204/7" value="47"/>
-<part name="R17" library="rcl" deviceset="R-EU_" device="0204/7" value="47"/>
-<part name="R18" library="rcl" deviceset="R-EU_" device="0204/7" value="560"/>
-<part name="R19" library="rcl" deviceset="R-EU_" device="0204/7" value="560"/>
+<part name="R15" library="rcl" deviceset="R-EU_" device="0207/10" value="120"/>
+<part name="R16" library="rcl" deviceset="R-EU_" device="0207/10" value="47"/>
+<part name="R17" library="rcl" deviceset="R-EU_" device="0207/10" value="47"/>
+<part name="R18" library="rcl" deviceset="R-EU_" device="0207/10" value="560"/>
+<part name="R19" library="rcl" deviceset="R-EU_" device="0207/10" value="560"/>
 <part name="GND16" library="supply1" deviceset="GND" device=""/>
 <part name="GND22" library="supply1" deviceset="GND" device=""/>
 <part name="+3V13" library="supply1" deviceset="+3V3" device=""/>
 <part name="GND23" library="supply1" deviceset="GND" device=""/>
-<part name="R20" library="rcl" deviceset="R-EU_" device="0204/7" value="560"/>
-<part name="C4" library="rcl" deviceset="CPOL-EU" device="SANYO_C"/>
+<part name="R20" library="rcl" deviceset="R-EU_" device="0207/10" value="560"/>
+<part name="C4" library="rcl" deviceset="CPOL-EU" device="E3.5-8"/>
 <part name="C6" library="rcl" deviceset="C-EU" device="C0805" value="0.1"/>
 </parts>
