File: sortirovka.sch (EAGLE design)
At the start: 72 parts, among them IC1 DS1307Z, IC3 LM1117IMPX-3.3, U1 MAX3485CSA, X1 PI3-CON, X10 MKDSN1,5/3-5,08, X3 MKDSN1,5/4-5,08, X4 MKDSN1,5/2-5,08, X5 22-23-2021, X6 22-23-2051, X7 22-23-2041, X8 22-23-2051, X9 MKDSN1,5/7-5,08

Commit message: rev 1.1 to produce
Parts:
- removed JP2: (no value), pinhead:PINHD-1X1
- OC1, OC10, OC2, OC3, OC4, OC5, OC6, OC7, OC8, OC9: device MyLib:SFH6106 -> MyLib:SFH6106REAL
- R16, R17: value 47 -> 15
- R18, R19: value 560 -> 1k5
- R20: value 560 -> 10
Connections:
- net N$43: no longer JP2.1
Changed lines of the file:
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@@
 <part name="R3" library="rcl" deviceset="R-EU_" device="R0805" value="200"/>
 <part name="R4" library="rcl" deviceset="R-EU_" device="R0805" value="200"/>
-<part name="OC1" library="MyLib" deviceset="SFH6106" device=""/>
-<part name="OC2" library="MyLib" deviceset="SFH6106" device=""/>
+<part name="OC1" library="MyLib" deviceset="SFH6106" device="REAL"/>
+<part name="OC2" library="MyLib" deviceset="SFH6106" device="REAL"/>
 <part name="R5" library="rcl" deviceset="R-EU_" device="R0805" value="10k"/>
 <part name="GND5" library="supply1" deviceset="GND" device=""/>
@@
 <part name="SUPPLY4" library="supply2" deviceset="GND1" device=""/>
 <part name="SUPPLY5" library="supply2" deviceset="GND1" device=""/>
-<part name="OC3" library="MyLib" deviceset="SFH6106" device=""/>
+<part name="OC3" library="MyLib" deviceset="SFH6106" device="REAL"/>
 <part name="R8" library="rcl" deviceset="R-EU_" device="R0805" value="10k"/>
 <part name="GND3" library="supply1" deviceset="GND" device=""/>
@@
 <part name="U$4" library="MyLib" deviceset="NSI45020AT1G" device="SOD-123"/>
 <part name="SUPPLY6" library="supply2" deviceset="GND1" device=""/>
-<part name="OC4" library="MyLib" deviceset="SFH6106" device=""/>
+<part name="OC4" library="MyLib" deviceset="SFH6106" device="REAL"/>
 <part name="R9" library="rcl" deviceset="R-EU_" device="R0805" value="10k"/>
 <part name="GND4" library="supply1" deviceset="GND" device=""/>
@@
 <part name="U$5" library="MyLib" deviceset="NSI45020AT1G" device="SOD-123"/>
 <part name="SUPPLY7" library="supply2" deviceset="GND1" device=""/>
-<part name="OC5" library="MyLib" deviceset="SFH6106" device=""/>
+<part name="OC5" library="MyLib" deviceset="SFH6106" device="REAL"/>
 <part name="R12" library="rcl" deviceset="R-EU_" device="R0805" value="10k"/>
 <part name="GND7" library="supply1" deviceset="GND" device=""/>
@@
 <part name="D9" library="MyLib" deviceset="DIODE" device="1N4007"/>
 <part name="SUPPLY13" library="supply2" deviceset="GND1" device=""/>
-<part name="OC6" library="MyLib" deviceset="SFH6106" device=""/>
+<part name="OC6" library="MyLib" deviceset="SFH6106" device="REAL"/>
 <part name="R13" library="rcl" deviceset="R-EU_" device="R0805" value="10k"/>
 <part name="GND8" library="supply1" deviceset="GND" device=""/>
@@
 <part name="D10" library="MyLib" deviceset="DIODE" device="1N4007"/>
 <part name="SUPPLY15" library="supply2" deviceset="GND1" device=""/>
-<part name="OC7" library="MyLib" deviceset="SFH6106" device=""/>
+<part name="OC7" library="MyLib" deviceset="SFH6106" device="REAL"/>
 <part name="GND2" library="supply1" deviceset="GND" device=""/>
 <part name="P+3" library="supply1" deviceset="+24V" device=""/>
-<part name="OC8" library="MyLib" deviceset="SFH6106" device=""/>
+<part name="OC8" library="MyLib" deviceset="SFH6106" device="REAL"/>
 <part name="GND9" library="supply1" deviceset="GND" device=""/>
 <part name="P+4" library="supply1" deviceset="+24V" device=""/>
-<part name="OC9" library="MyLib" deviceset="SFH6106" device=""/>
+<part name="OC9" library="MyLib" deviceset="SFH6106" device="REAL"/>
 <part name="GND12" library="supply1" deviceset="GND" device=""/>
 <part name="P+5" library="supply1" deviceset="+24V" device=""/>
-<part name="OC10" library="MyLib" deviceset="SFH6106" device=""/>
+<part name="OC10" library="MyLib" deviceset="SFH6106" device="REAL"/>
 <part name="GND13" library="supply1" deviceset="GND" device=""/>
 <part name="P+6" library="supply1" deviceset="+24V" device=""/>
-<part name="JP2" library="pinhead" deviceset="PINHD-1X1" device=""/>
 <part name="+3V11" library="supply1" deviceset="+3V3" device=""/>
 <part name="GND24" library="supply1" deviceset="GND" device=""/>
@@
 <part name="C3" library="rcl" deviceset="C-EU" device="C0805" value="0.1"/>
 <part name="R15" library="rcl" deviceset="R-EU_" device="0207/10" value="120"/>
-<part name="R16" library="rcl" deviceset="R-EU_" device="0207/10" value="47"/>
-<part name="R17" library="rcl" deviceset="R-EU_" device="0207/10" value="47"/>
-<part name="R18" library="rcl" deviceset="R-EU_" device="0207/10" value="560"/>
-<part name="R19" library="rcl" deviceset="R-EU_" device="0207/10" value="560"/>
+<part name="R16" library="rcl" deviceset="R-EU_" device="0207/10" value="15"/>
+<part name="R17" library="rcl" deviceset="R-EU_" device="0207/10" value="15"/>
+<part name="R18" library="rcl" deviceset="R-EU_" device="0207/10" value="1k5"/>
+<part name="R19" library="rcl" deviceset="R-EU_" device="0207/10" value="1k5"/>
 <part name="GND16" library="supply1" deviceset="GND" device=""/>
 <part name="GND22" library="supply1" deviceset="GND" device=""/>
 <part name="+3V13" library="supply1" deviceset="+3V3" device=""/>
 <part name="GND23" library="supply1" deviceset="GND" device=""/>
-<part name="R20" library="rcl" deviceset="R-EU_" device="0207/10" value="560"/>
+<part name="R20" library="rcl" deviceset="R-EU_" device="0207/10" value="10"/>
 <part name="C4" library="rcl" deviceset="CPOL-EU" device="E3.5-8"/>
 <part name="C6" library="rcl" deviceset="C-EU" device="C0805" value="0.1"/>
@@
 <instance part="GND13" gate="1" x="269.24" y="2.54"/>
 <instance part="P+6" gate="1" x="287.02" y="17.78"/>
-<instance part="JP2" gate="G$1" x="45.72" y="50.8"/>
 <instance part="+3V11" gate="G$1" x="43.18" y="154.94"/>
 <instance part="GND24" gate="1" x="299.72" y="124.46"/>
@@
 </segment>
 </net>
-<net name="N$23" class="0">
-<segment>
-<pinref part="Q5" gate="G$1" pin="1"/>
-<pinref part="IC1" gate="G$1" pin="X1"/>
-<wire x1="35.56" y1="139.7" x2="45.72" y2="139.7" width="0.1524" layer="91"/>
-</segment>
-</net>
-<net name="N$25" class="0">
-<segment>
-<pinref part="IC1" gate="G$1" pin="X2"/>
-<pinref part="Q5" gate="G$1" pin="2"/>
-<wire x1="45.72" y1="134.62" x2="35.56" y2="134.62" width="0.1524" layer="91"/>
-</segment>
-</net>
 <net name="N$4" class="0">
 <segment>
@@
 <wire x1="38.1" y1="58.42" x2="38.1" y2="50.8" width="0.1524" layer="91"/>
 <wire x1="38.1" y1="50.8" x2="12.7" y2="50.8" width="0.1524" layer="91"/>
-<pinref part="JP2" gate="G$1" pin="1"/>
-<wire x1="38.1" y1="50.8" x2="43.18" y2="50.8" width="0.1524" layer="91"/>
 </segment>
 </net>
@@
 </segment>
 </net>
+<net name="N$23" class="0">
+<segment>
+<pinref part="IC1" gate="G$1" pin="X1"/>
+<pinref part="Q5" gate="G$1" pin="1"/>
+<wire x1="45.72" y1="139.7" x2="35.56" y2="139.7" width="0.1524" layer="91"/>
+</segment>
+</net>
+<net name="N$25" class="0">
+<segment>
+<pinref part="Q5" gate="G$1" pin="2"/>
+<pinref part="IC1" gate="G$1" pin="X2"/>
+<wire x1="35.56" y1="134.62" x2="45.72" y2="134.62" width="0.1524" layer="91"/>
+</segment>
+</net>

Commit message: manufacture-1
Parts:
- R12, R13, R5, R6, R8, R9: value 10k -> 1k

Commit message: wip
Parts:
- added Q1: (no value), MyLib:IRLMS6702PBF
Connections:
- new net N$48: Q1.D@1, Q1.D@2, Q1.D@3, Q1.D@4, X5-1.S
- net GND: now also Q1.G
- net PW: now also Q1.S; no longer X5-1.S
Other:
- moved on the sheet: X5-1, X5-2
Changed lines of the file:
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@@
 <part name="C4" library="rcl" deviceset="CPOL-EU" device="E3.5-8"/>
 <part name="C6" library="rcl" deviceset="C-EU" device="C0805" value="0.1"/>
+<part name="Q1" library="MyLib" deviceset="IRLMS6702PBF" device=""/>
 </parts>
 <sheets>
@@
 <plain>
 <text x="48.26" y="121.92" size="1.778" layer="91">(PCF85263A)</text>
-<text x="299.72" y="66.04" size="1.778" layer="91">B(-)</text>
-<text x="299.72" y="76.2" size="1.778" layer="91">A(+)</text>
+<text x="299.72" y="66.04" size="1.778" layer="91">A(+)</text>
+<text x="299.72" y="78.74" size="1.778" layer="91">B(-)</text>
 </plain>
 <instances>
@@
 <instance part="IC3" gate="G$1" x="218.44" y="129.54"/>
 <instance part="+3V12" gate="G$1" x="243.84" y="137.16"/>
-<instance part="X5" gate="-1" x="187.96" y="129.54" rot="R180"/>
-<instance part="X5" gate="-2" x="187.96" y="121.92" rot="R180"/>
+<instance part="X5" gate="-1" x="167.64" y="129.54" rot="R180"/>
+<instance part="X5" gate="-2" x="167.64" y="121.92" rot="R180"/>
 <instance part="GND21" gate="1" x="190.5" y="119.38"/>
 <instance part="C5" gate="G$1" x="294.64" y="132.08"/>
@@
 <instance part="C4" gate="G$1" x="276.86" y="-68.58"/>
 <instance part="C6" gate="G$1" x="281.94" y="-68.58"/>
+<instance part="Q1" gate="G$1" x="177.8" y="129.54" rot="MR90"/>
 </instances>
 <busses>
@@
 </segment>
 <segment>
-<pinref part="X5" gate="-2" pin="S"/>
 <pinref part="GND21" gate="1" pin="GND"/>
-<junction x="190.5" y="121.92"/>
 <pinref part="GND21" gate="1" pin="GND"/>
 <pinref part="C2" gate="G$1" pin="-"/>
 <pinref part="C3" gate="G$1" pin="2"/>
 <wire x1="190.5" y1="121.92" x2="203.2" y2="121.92" width="0.1524" layer="91"/>
+<junction x="190.5" y="121.92"/>
+<pinref part="X5" gate="-2" pin="S"/>
+<wire x1="170.18" y1="121.92" x2="180.34" y2="121.92" width="0.1524" layer="91"/>
+<wire x1="180.34" y1="121.92" x2="190.5" y2="121.92" width="0.1524" layer="91"/>
+<wire x1="180.34" y1="124.46" x2="180.34" y2="121.92" width="0.1524" layer="91"/>
+<junction x="180.34" y="121.92"/>
+<pinref part="Q1" gate="G$1" pin="G"/>
 </segment>
 <segment>
@@
 <pinref part="R16" gate="G$1" pin="2"/>
 <pinref part="R18" gate="G$1" pin="2"/>
-<wire x1="251.46" y1="60.96" x2="251.46" y2="63.5" width="0.1524" layer="91"/>
-<wire x1="251.46" y1="63.5" x2="251.46" y2="73.66" width="0.1524" layer="91"/>
-<wire x1="251.46" y1="73.66" x2="274.32" y2="73.66" width="0.1524" layer="91"/>
+<wire x1="256.54" y1="60.96" x2="256.54" y2="73.66" width="0.1524" layer="91"/>
+<wire x1="256.54" y1="73.66" x2="274.32" y2="73.66" width="0.1524" layer="91"/>
 <pinref part="U$3" gate="G$1" pin="P$1"/>
-<wire x1="256.54" y1="60.96" x2="251.46" y2="60.96" width="0.1524" layer="91"/>
 <pinref part="U1" gate="G$1" pin="B"/>
-<wire x1="236.22" y1="63.5" x2="251.46" y2="63.5" width="0.1524" layer="91"/>
+<wire x1="236.22" y1="63.5" x2="241.3" y2="63.5" width="0.1524" layer="91"/>
+<wire x1="241.3" y1="63.5" x2="241.3" y2="73.66" width="0.1524" layer="91"/>
+<wire x1="241.3" y1="73.66" x2="256.54" y2="73.66" width="0.1524" layer="91"/>
+<junction x="256.54" y="73.66"/>
 </segment>
 </net>
@@
 <net name="PW" class="0">
 <segment>
-<pinref part="X5" gate="-1" pin="S"/>
 <pinref part="IC3" gate="G$1" pin="IN"/>
 <wire x1="210.82" y1="129.54" x2="203.2" y2="129.54" width="0.1524" layer="91"/>
 <label x="198.12" y="129.54" size="1.778" layer="95"/>
+<pinref part="C3" gate="G$1" pin="1"/>
 <pinref part="C2" gate="G$1" pin="+"/>
-<junction x="190.5" y="129.54"/>
-<pinref part="C3" gate="G$1" pin="1"/>
+<wire x1="182.88" y1="129.54" x2="190.5" y2="129.54" width="0.1524" layer="91"/>
 <wire x1="203.2" y1="129.54" x2="190.5" y2="129.54" width="0.1524" layer="91"/>
-<junction x="203.2" y="129.54"/>
+<pinref part="Q1" gate="G$1" pin="S"/>
 </segment>
 <segment>
@@
 <pinref part="U1" gate="G$1" pin="A"/>
 <wire x1="236.22" y1="60.96" x2="246.38" y2="60.96" width="0.1524" layer="91"/>
-<wire x1="246.38" y1="60.96" x2="246.38" y2="66.04" width="0.1524" layer="91"/>
-<wire x1="246.38" y1="66.04" x2="261.62" y2="66.04" width="0.1524" layer="91"/>
-<wire x1="261.62" y1="66.04" x2="261.62" y2="63.5" width="0.1524" layer="91"/>
+<wire x1="246.38" y1="60.96" x2="246.38" y2="63.5" width="0.1524" layer="91"/>
+<wire x1="246.38" y1="63.5" x2="261.62" y2="63.5" width="0.1524" layer="91"/>
+<junction x="261.62" y="63.5"/>
 </segment>
 </net>
@@
 </segment>
 </net>
+<net name="N$48" class="0">
+<segment>
+<pinref part="X5" gate="-1" pin="S"/>
+<wire x1="170.18" y1="129.54" x2="172.72" y2="129.54" width="0.1524" layer="91"/>
+<pinref part="Q1" gate="G$1" pin="D@1"/>
+<pinref part="Q1" gate="G$1" pin="D@2"/>
+<junction x="172.72" y="129.54"/>
+<pinref part="Q1" gate="G$1" pin="D@3"/>
+<pinref part="Q1" gate="G$1" pin="D@4"/>
+</segment>
+</net>

Commit message: wip
Parts:
- removed R12, R13, R5, R6, R8, R9: 1k, rcl:R-EU_R0805
- removed R14, R7: 0, rcl:R-EU_R0805
- removed R16, R17: 15, rcl:R-EU_0207/10
- removed R18, R19: 1k5, rcl:R-EU_0207/10
- removed R20: 10, rcl:R-EU_0207/10
- removed X10: MKDSN1,5/3-5,08, con-phoenix-508:MKDSN1,5/3-5,08
- added C11, C12: (no value), rcl:C-EUC0805
- added C13, C20: 10uF, rcl:C-EUC0805
- added C14, C16, C18, C19: 100nF, rcl:C-EUC0805
- added C15, C17: 10nF, rcl:C-EUC0805
- added D11: CDSOT23-SM712SOT23-R, MyLib:CDSOT23-SM712SOT23-R
- added D12, D13: DIODE1N4007, MyLib:DIODE1N4007
- added GDT1, GDT2: GDT-2031-XXT-SM, supressor:GDT-2031-XXT-SM
- added IC2: MEGA8-AI, atmel:MEGA8-AI
- added IC4, IC5: PCF8574T, micro-philips:PCF8574T
- added IC6: MEGA32-A, atmel:MEGA32-A
- added JP1: (no value), pinhead:PINHD-1X9/90
- added JP4: (no value), pinhead:PINHD-2X3
- added L1, L2: (no value), rcl:L-US0402
- added OC11, OC12: (no value), MyLib:SFH6106REAL
- added Q2: (no value), crystal:CRYSTALSM49
- added U$8: NSI45020AT1GSOD-123, MyLib:NSI45020AT1GSOD-123
- added Z1, Z2: TBU-CA, supressor:TBU-CA
- R1, R2, R3, R4: value 200 -> 50
- R15: value 120 -> 1k; device rcl:R-EU_0207/10 -> rcl:R-EU_R0805
- U$3: value NUP2105LSOT23-R -> NSI45020AT1GSOD-123; device MyLib:NUP2105LSOT23-R -> MyLib:NSI45020AT1GSOD-123
- U1: value MAX3485CSA -> ADM2587EBRWZ; device MyLib:RS485SOIC -> Analog Devices_By_element14_Batch_1:ADM2587EBRWZ
- X1: value PI3-CON -> MKDSN1,5/3-5,08; device MyLib:PI3-CON -> MyLib:MKDSN1,5/3-5,08
Connections:
- removed net N$43: OC1.EMIT, R5.2, X1.GPIO04
- new net +5V: JP4.2
- new net A: D11.P$1, U1.A, Z1.2
- new net B: D11.P$2, U1.B, Z2.2
- new net INT-S: IC4.P0, IC5.!INT
- new net INT0: IC2.PD2(INT0), IC4.!INT
- new net N$49: IC4.P4, JP1.5
- new net N$50: IC4.P3, JP1.6
- new net N$51: IC4.P2, JP1.7
- new net N$52: IC4.P1, JP1.9
- new net N$53: JP1.8, R15.1
- new net N$54: IC5.P7, OC1.COL
- new net N$55: IC5.P6, OC2.COL
- new net N$56: IC5.P5, OC3.COL
- new net N$57: IC5.P4, OC4.COL
- new net N$58: IC5.P3, OC5.COL
- new net PE: C13.2, C15.2, C16.2, D11.P$3, GDT1.1, GDT2.2, L2.2, U1.GND2, U1.GND2_2, X1-2.KL
- new net R/W: IC2.PB0(ICP), U1.DE, U1.~RE
- new net RESET: IC2.PC6(/RESET), JP4.5
- new net RS2: IC2.PD3(INT1)
- new net RXD: IC2.PD0(RXD), U1.RXD
- new net SCK: IC2.PB5(SCK), JP4.3
- new net SCL: IC1.SCL, IC2.PC5(ADC5/SCL), IC4.SCL, IC5.SCL, R10.1, X7-3.S
- new net SDA: IC1.SDA, IC2.PC4(ADC4/SDA), IC4.SDA, IC5.SDA, R11.1, X7-2.S
- new net TXD: IC2.PD1(TXD), U1.TXD
- new net VCC: C17.1, C18.1, C19.1, C20.1, U1.VCC, U1.VCC_2
- net +3V3: now also IC4.VDD, IC5.A0, IC5.VDD, R15.2; no longer OC1.COL, OC2.COL, OC3.COL, OC4.COL, OC5.COL, OC6.COL, R19.2, R7.2, U1.VCC
- net GND: now also C11.2, C12.1, C17.2, C18.2, C19.2, C20.2, IC4.A0, IC4.A1, IC4.A2, IC4.VSS, IC5.A1, IC5.A2, IC5.VSS, JP1.1, JP4.6, OC1.EMIT, OC11.EMIT, OC12.EMIT, OC2.EMIT, OC3.EMIT, OC4.EMIT, OC5.EMIT, OC6.EMIT, U1.GND1, U1.GND1_2, U1.GND1_3, U1.GND1_4; no longer R12.1, R13.1, R18.1, R20.2, R5.1, R6.1, R8.1, R9.1, U$3.P$3, U1.GND, X1.GND@1, X1.GND@2, X1.GND@3, X1.GND@4, X1.GND@5, X1.GND@6, X1.GND@7, X1.GND@8
- net GND1: now also D12.A, D13.A, OC11.C, OC12.C
- net MISO: now also IC2.PB4(MISO), JP4.1; no longer X1.GPIO09
- net MOSI: now also IC2.PB3(MOSI/OC2), JP4.4; no longer X1.GPIO10
- net N$1: now also GDT1.2, X1-1.KL, Z1.1; no longer U1.DI, X1.GPIO14
- net N$14: now also C11.1, IC2.PB7(XTAL2/TOSC2), Q2.1; no longer R7.1, X1.3.3V@1, X1.3.3V@2
- net N$2: now also GDT2.1, X1-3.KL, Z2.1; no longer U1.RO, X1.GPIO15
- net N$26: now also C12.2, IC2.PB6(XTAL1/TOSC1), Q2.2; no longer IC1.SCL, R10.1, X1.GPIO03, X7-3.S
- net N$27: now also D12.C, OC11.A, U$3.C; no longer IC1.SDA, R11.1, X1.GPIO02, X7-2.S
- net N$28: now also U$3.A; no longer R14.1, X1.+5V@1, X1.+5V@2
- net N$3: now also C13.1, C15.1, C16.1, L1.2, U1.VISOIN; no longer U1./RE, U1.DE, X1.GPIO18
- net N$34: now also D13.C, OC12.A, U$8.C; no longer OC6.EMIT, R13.2, X1.GPIO26
- net N$39: now also U$8.A; no longer OC5.EMIT, R12.2, X1.GPIO19
- net N$4: now also C14.2, L2.1, U1.GND2_3, U1.GND2_4; no longer R16.2, R18.2, U$3.P$1, U1.B
- net N$40: now also IC5.P2, OC6.COL; no longer OC4.EMIT, R9.2, X1.GPIO13
- net N$41: now also IC5.P1, OC11.COL; no longer OC3.EMIT, R8.2, X1.GPIO06
- net N$42: now also IC5.P0, OC12.COL; no longer OC2.EMIT, R6.2, X1.GPIO05
- net N$45: now also IC4.P7, JP1.2; no longer R15.2, R16.1, X10-2.KL
- net N$46: now also IC4.P6, JP1.3; no longer R15.1, R17.1, X10-1.KL
- net N$47: now also IC4.P5, JP1.4; no longer R17.2, R19.1, U$3.P$2, U1.A
- net N$5: now also C14.1, L1.1, U1.VISOOUT; no longer R20.1, X10-3.KL
- net N$6: now also IC2.PC0(ADC0), R4.2; no longer R1.2, X1.GPIO21
- net N$7: now also IC2.PC1(ADC1), R3.2; no longer R2.2, X1.GPIO20
- net N$8: now also IC2.PC2(ADC2), R2.2; no longer R3.2, X1.GPIO16
- net N$9: now also IC2.PC3(ADC3), R1.2; no longer R4.2, X1.GPIO12
- net PW: no longer R14.2
- net SPI0: no longer X1.GPIO08
- net SPI1: no longer X1.GPIO07
- net SPI_CLK: no longer X1.GPIO11
Other:
- note removed: "A(+)"
- note removed: "B(-)"
- moved on the sheet: R1, R15, R2, R3, R4
