File: sortirovka.sch (EAGLE design)
At the start: 87 parts, among them IC1 DS1307Z, IC2 MEGA8-AI, IC3 LM1117IMPX-3.3, IC4 PCF8574T, IC5 PCF8574T, IC6 MEGA32-A, U1 ADM2587EBRWZ, X1 MKDSN1,5/3-5,08, X3 MKDSN1,5/4-5,08, X4 MKDSN1,5/2-5,08, X5 22-23-2021, X6 22-23-2051, X7 22-23-2041, X8 22-23-2051, X9 MKDSN1,5/7-5,08

Commit message: main pars on the board
Parts:
- removed Q1: (no value), MyLib:IRLMS6702PBF
- removed X8: 22-23-2051, con-molex:22-23-2051
- added J1: ATTEND-MICROSD-112, sd-mmc:ATTEND-MICROSD-112
- added R12, R5, R6: 3.3k, rcl:R-EU_M0805
- added R13: 100k, rcl:R-EU_M0805
- added R7, R8, R9: 1.8k, rcl:R-EU_M0805
- added U$10: 2X16LCDBOTH, MyLib:2X16LCDBOTH
- added U$9: W5100_MODULESMALL, MyLib:W5100_MODULESMALL
- IC6: value MEGA32-A -> PCF8574T; device atmel:MEGA32-A -> micro-philips:PCF8574T
- JP1: device pinhead:PINHD-1X9/90 -> pinhead:PINHD-1X9
Connections:
- removed net PW: C2.+, C3.1, IC3.IN, Q1.S
- removed net SPI1: X8-4.S
- removed net VCC: C17.1, C18.1, C19.1, C20.1, U1.VCC, U1.VCC_2
- new net E_RESET: U$9.RESET
- new net E_SELECT: U$9.SS
- new net ID0: IC6.P4, U$10.D0
- new net ID1: IC6.P5, U$10.D1
- new net ID2: IC6.P6, U$10.D2
- new net ID3: IC6.P7, U$10.D3
- new net I_E: IC6.P3, U$10.E
- new net I_RS: IC6.P1, U$10.RS
- new net I_RW: IC6.P2, U$10.RW
- new net N$43: J1.CD/DAT3(!CS!), R12.2, R9.1
- new net N$59: J1.CMD(DI), R6.2, R8.1
- new net N$60: J1.CLK(SCLK), R5.2, R7.1
- new net N$61: IC6.SCL
- new net N$73: U$10.VO
- new net SD_DETECT: J1.CD, R13.1
- new net SD_SELECT: R9.2
- net +3V3: now also J1.VDD, R13.2; no longer IC1.VCC, IC4.VDD, IC5.A0, IC5.VDD, R10.2, R11.2, R15.2, X7-1.S
- net +5V: now also C17.1, C18.1, C19.1, C2.+, C20.1, C3.1, IC1.VCC, IC3.IN, IC4.VDD, IC5.A0, IC5.VDD, IC6.A1, IC6.VDD, R10.2, R11.2, R15.2, U$10.VDD, U$9.VCC, U1.VCC, U1.VCC_2, X5-1.S, X7-1.S
- net GND: now also IC6.A0, IC6.A2, IC6.VSS, J1.GND, J1.S@1, J1.S@2, J1.VSS(GND), R12.1, R5.1, R6.1, U$10.VSS, U$9.GND@1; no longer Q1.G, X8-5.S
- net MISO: now also J1.DAT0(DO), U$9.MISO; no longer X8-2.S
- net MOSI: now also R8.2, U$9.MOSI; no longer X8-3.S
- net N$48: now also IC6.SDA; no longer Q1.D@1, Q1.D@2, Q1.D@3, Q1.D@4, X5-1.S
- net SCK: now also R7.2, U$9.SCK
- net SPI_CLK: no longer X8-1.S

Commit message: wip
Parts:
- removed D3: DIODE1N4007, MyLib:DIODE1N4007
- removed X9: MKDSN1,5/7-5,08, con-phoenix-508:MKDSN1,5/7-5,08
- added D14: BAV199, MyLib:BAV199
- added IC7: PCF8574T, micro-philips:PCF8574T
- added U$11, U$12, U$13, U$14: NSI45020AT1GSOD-123, MyLib:NSI45020AT1GSOD-123
- added U2: TRACO_TEL_5-1211, MyLib:TRACO_TEL_5-1211
- added X2, X8: MKDSN1,5/4-5,08, con-phoenix-508:MKDSN1,5/4-5,08
- C1, C2, C4: device rcl:CPOL-EUE3.5-8 -> rcl:CPOL-EU153CLV-0605
- D1, D10, D12, D13, D2, D4, D5, D6, D7, D8, D9: value DIODE1N4007 -> BAV199; device MyLib:DIODE1N4007 -> MyLib:BAV199
Connections:
- net N$73 renamed I_CONTRAST
- net R/W renamed 485_R/W
- removed net ID0: IC6.P4, U$10.D0
- removed net ID1: IC6.P5, U$10.D1
- removed net ID2: IC6.P6, U$10.D2
- removed net ID3: IC6.P7, U$10.D3
- removed net N$52: IC4.P1, JP1.9
- removed net N$61: IC6.SCL
- removed net PE: C13.2, C15.2, C16.2, D11.P$3, GDT1.1, GDT2.2, L2.2, U1.GND2, U1.GND2_2, X1-2.KL
- removed net RS2: IC2.PD3(INT1)
- removed net SPI_CLK: X6-1.S
- new net INT1: IC2.PD3(INT1), IC5.!INT
- new net I_D0: IC7.P0, U$10.D0
- new net I_D1: IC7.P1, U$10.D1
- new net I_D2: IC7.P2, U$10.D2
- new net I_D3: IC7.P3, U$10.D3
- new net I_D4: IC7.P4, U$10.D4
- new net I_D5: IC7.P5, U$10.D5
- new net I_D6: IC7.P6, U$10.D6
- new net I_D7: IC7.P7, U$10.D7
- new net N$62: U$11.C, X3-1.KL
- new net N$63: U$12.C, X3-2.KL
- new net N$65: U$13.C, X3-3.KL
- new net N$67: U$14.C, X3-4.KL
- net +24V: now also D1.C, D10.C, D12.C, D13.C, D14.C, D2.C, D4.C, D5.C, D6.C, D7.C, D8.C, D9.C, U2.+VIN@1, U2.+VIN@2
- net +3V3: no longer C10.1, C8.1, C9.1
- net +5V: now also C10.1, C8.1, C9.1, IC2.VCC@1, IC2.VCC@2, IC7.A0, IC7.A1, IC7.VDD, U2.+VOUT
- net E_SELECT: now also IC2.PB2(SS/OC1B)
- net GND: now also IC2.GND@1, IC2.GND@2, IC7.A2, IC7.VSS, U2.-V0UT
- net GND1: now also C13.2, C15.2, C16.2, D11.P$3, D14.A, GDT1.1, GDT2.2, L2.2, U1.GND2, U1.GND2_2, U2.-VIN@1, U2.-VIN@2, X1-2.KL; no longer D3.A, X9-1.KL
- net INT-S: no longer IC5.!INT
- net I_E: now also IC6.P5; no longer IC6.P3
- net I_RS: now also IC6.P7; no longer IC6.P1
- net I_RW: now also IC6.P6; no longer IC6.P2
- net N$10: now also D13.AC, U$11.A; no longer D4.C, X3-1.KL
- net N$11: now also D4.AC, U$12.A; no longer D1.C, X3-2.KL
- net N$12: now also D1.AC, U$13.A; no longer D2.C, X3-3.KL
- net N$13: now also D2.AC, U$14.A; no longer D3.C, X3-4.KL
- net N$16: now also D14.AC; no longer D5.C
- net N$17: now also D5.AC; no longer D6.C
- net N$21: now also X2-4.KL; no longer X9-7.KL
- net N$22: now also X2-3.KL; no longer X9-6.KL
- net N$24: now also D6.AC; no longer D7.C
- net N$27: now also D7.AC, OC4.A, U$5.C; no longer D12.C, OC11.A, U$3.C
- net N$28: now also X8-2.KL
- net N$30: now also D8.AC, OC5.A, U$6.C; no longer D8.C, OC4.A, U$5.C
- net N$32: now also D9.AC, OC6.A, U$7.C; no longer D9.C, OC5.A, U$6.C
- net N$33: now also X2-1.KL; no longer X9-4.KL
- net N$34: now also D10.AC, OC11.A, U$3.C; no longer D13.C, OC12.A, U$8.C
- net N$35: now also X2-2.KL; no longer X9-5.KL
- net N$36: now also D12.AC, OC12.A, U$8.C; no longer D10.C, OC6.A, U$7.C
- net N$37: now also X8-4.KL; no longer X9-3.KL
- net N$38: now also X8-3.KL; no longer X9-2.KL
- net N$39: now also X8-1.KL
- net N$48: now also IC4.P1, JP1.6; no longer IC6.SDA
- net N$50: now also JP1.9; no longer JP1.6
- net SCK: now also X6-1.S
- net SCL: now also IC6.SCL, IC7.SCL
- net SDA: now also IC6.SDA, IC7.SDA
- net SD_SELECT: now also IC2.PD5(T1)
Other:
- moved on the sheet: C10, C4, C6, C8, C9, IC6, X3-1, X3-2, X3-3, X3-4, X4-1, X4-2

Commit message: All routed.
Connections:
- net N$21: now also X2-1.KL; no longer X2-4.KL
- net N$22: now also X2-2.KL; no longer X2-3.KL
- net N$28: now also X8-3.KL; no longer X8-2.KL
- net N$33: now also X2-4.KL; no longer X2-1.KL
- net N$35: now also X2-3.KL; no longer X2-2.KL
- net N$37: now also X8-1.KL; no longer X8-4.KL
- net N$38: now also X8-2.KL; no longer X8-3.KL
- net N$39: now also X8-4.KL; no longer X8-1.KL
Other:
- moved on the sheet: X2-1, X2-2, X2-3, X2-4, X8-1, X8-2, X8-3, X8-4
Changed lines of the file:
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@@
 <instance part="GND39" gate="1" x="190.5" y="81.28"/>
 <instance part="P+23" gate="1" x="190.5" y="111.76"/>
-<instance part="X2" gate="-1" x="-76.2" y="22.86" rot="R180"/>
-<instance part="X2" gate="-2" x="-76.2" y="27.94" rot="R180"/>
-<instance part="X2" gate="-3" x="-76.2" y="33.02" rot="R180"/>
-<instance part="X2" gate="-4" x="-76.2" y="38.1" rot="R180"/>
-<instance part="X8" gate="-1" x="-76.2" y="-152.4" rot="R180"/>
-<instance part="X8" gate="-2" x="-76.2" y="-147.32" rot="R180"/>
-<instance part="X8" gate="-3" x="-76.2" y="-142.24" rot="R180"/>
-<instance part="X8" gate="-4" x="-76.2" y="-137.16" rot="R180"/>
+<instance part="X2" gate="-1" x="-88.9" y="38.1" rot="R180"/>
+<instance part="X2" gate="-2" x="-88.9" y="33.02" rot="R180"/>
+<instance part="X2" gate="-3" x="-88.9" y="27.94" rot="R180"/>
+<instance part="X2" gate="-4" x="-88.9" y="22.86" rot="R180"/>
+<instance part="X8" gate="-1" x="-91.44" y="-137.16" rot="R180"/>
+<instance part="X8" gate="-2" x="-91.44" y="-142.24" rot="R180"/>
+<instance part="X8" gate="-3" x="-91.44" y="-147.32" rot="R180"/>
+<instance part="X8" gate="-4" x="-91.44" y="-152.4" rot="R180"/>
 <instance part="D14" gate="G$1" x="-7.62" y="55.88" rot="R270"/>
 <instance part="P+24" gate="1" x="-7.62" y="68.58" rot="MR0"/>
@@
 <pinref part="U$2" gate="G$1" pin="A"/>
 <wire x1="-45.72" y1="25.4" x2="-35.56" y2="25.4" width="0.1524" layer="91"/>
-<pinref part="X2" gate="-3" pin="KL"/>
-<wire x1="-73.66" y1="33.02" x2="-45.72" y2="33.02" width="0.1524" layer="91"/>
 <wire x1="-45.72" y1="33.02" x2="-45.72" y2="25.4" width="0.1524" layer="91"/>
+<pinref part="X2" gate="-2" pin="KL"/>
+<wire x1="-86.36" y1="33.02" x2="-45.72" y2="33.02" width="0.1524" layer="91"/>
 </segment>
 </net>
@@
 <wire x1="-35.56" y1="-10.16" x2="-50.8" y2="-10.16" width="0.1524" layer="91"/>
 <wire x1="-50.8" y1="-10.16" x2="-50.8" y2="27.94" width="0.1524" layer="91"/>
-<pinref part="X2" gate="-2" pin="KL"/>
-<wire x1="-50.8" y1="27.94" x2="-73.66" y2="27.94" width="0.1524" layer="91"/>
+<pinref part="X2" gate="-3" pin="KL"/>
+<wire x1="-50.8" y1="27.94" x2="-86.36" y2="27.94" width="0.1524" layer="91"/>
 </segment>
 </net>
@@
 <wire x1="-35.56" y1="-86.36" x2="-71.12" y2="-86.36" width="0.1524" layer="91"/>
 <wire x1="-71.12" y1="-86.36" x2="-71.12" y2="-137.16" width="0.1524" layer="91"/>
-<pinref part="X8" gate="-4" pin="KL"/>
-<wire x1="-71.12" y1="-137.16" x2="-73.66" y2="-137.16" width="0.1524" layer="91"/>
+<pinref part="X8" gate="-1" pin="KL"/>
+<wire x1="-71.12" y1="-137.16" x2="-88.9" y2="-137.16" width="0.1524" layer="91"/>
 </segment>
 </net>
@@
 <pinref part="U$5" gate="G$1" pin="A"/>
 <wire x1="-55.88" y1="-48.26" x2="-35.56" y2="-48.26" width="0.1524" layer="91"/>
-<pinref part="X2" gate="-1" pin="KL"/>
-<wire x1="-73.66" y1="22.86" x2="-55.88" y2="22.86" width="0.1524" layer="91"/>
 <wire x1="-55.88" y1="22.86" x2="-55.88" y2="-48.26" width="0.1524" layer="91"/>
+<pinref part="X2" gate="-4" pin="KL"/>
+<wire x1="-86.36" y1="22.86" x2="-55.88" y2="22.86" width="0.1524" layer="91"/>
 </segment>
 </net>
@@
 <pinref part="U$7" gate="G$1" pin="A"/>
 <wire x1="-35.56" y1="-127" x2="-66.04" y2="-127" width="0.1524" layer="91"/>
-<pinref part="X8" gate="-3" pin="KL"/>
-<wire x1="-73.66" y1="-142.24" x2="-66.04" y2="-142.24" width="0.1524" layer="91"/>
 <wire x1="-66.04" y1="-142.24" x2="-66.04" y2="-127" width="0.1524" layer="91"/>
+<pinref part="X8" gate="-2" pin="KL"/>
+<wire x1="-88.9" y1="-142.24" x2="-66.04" y2="-142.24" width="0.1524" layer="91"/>
 </segment>
 </net>
@@
 <wire x1="-35.56" y1="-167.64" x2="-63.5" y2="-167.64" width="0.1524" layer="91"/>
 <wire x1="-63.5" y1="-167.64" x2="-63.5" y2="-147.32" width="0.1524" layer="91"/>
-<pinref part="X8" gate="-2" pin="KL"/>
-<wire x1="-63.5" y1="-147.32" x2="-73.66" y2="-147.32" width="0.1524" layer="91"/>
+<pinref part="X8" gate="-3" pin="KL"/>
+<wire x1="-63.5" y1="-147.32" x2="-88.9" y2="-147.32" width="0.1524" layer="91"/>
 </segment>
 </net>
@@
 <pinref part="U$8" gate="G$1" pin="A"/>
 <wire x1="-35.56" y1="-208.28" x2="-68.58" y2="-208.28" width="0.1524" layer="91"/>
-<pinref part="X8" gate="-1" pin="KL"/>
-<wire x1="-73.66" y1="-152.4" x2="-68.58" y2="-152.4" width="0.1524" layer="91"/>
 <wire x1="-68.58" y1="-152.4" x2="-68.58" y2="-208.28" width="0.1524" layer="91"/>
+<pinref part="X8" gate="-4" pin="KL"/>
+<wire x1="-88.9" y1="-152.4" x2="-68.58" y2="-152.4" width="0.1524" layer="91"/>
 </segment>
 </net>
@@
 <wire x1="-35.56" y1="55.88" x2="-68.58" y2="55.88" width="0.1524" layer="91"/>
 <wire x1="-68.58" y1="55.88" x2="-68.58" y2="38.1" width="0.1524" layer="91"/>
-<pinref part="X2" gate="-4" pin="KL"/>
-<wire x1="-68.58" y1="38.1" x2="-73.66" y2="38.1" width="0.1524" layer="91"/>
-</segment>
-</net>
+<pinref part="X2" gate="-1" pin="KL"/>
+<wire x1="-68.58" y1="38.1" x2="-86.36" y2="38.1" width="0.1524" layer="91"/>
+</segment>
+</net>

Commit message: wip
Parts:
- added C21, C22: 0.1, rcl:C-EUC0805
Connections:
- net +5V: now also C21.1, C22.1
- net 485_R/W: now also IC2.PD4(XCK/T0); no longer IC2.PB0(ICP)
- net GND: now also C21.2, C22.2
- net SD_SELECT: now also IC2.PB1(OC1A); no longer IC2.PD5(T1)
Other:
- moved on the sheet: C1, C10, C2, C3, C4, C5, C6, C7, C8, C9, IC3, U2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

Commit message: Ready to gerber
Parts:
- added C23, C24, C25, C26: 0.1, rcl:C-EUC0805
- added IC8: DS1813-SMD, MyLib:DS1813-SMD
- added JP2: (no value), pinhead:PINHD-1X3
- added JP3: (no value), pinhead:PINHD-1X4
Connections:
- new net N$61: C23.1, IC2.AREF
- new net N$64: IC2.PD6(AIN0), JP3.3
- new net N$66: IC2.PD5(T1), JP3.4
- net +24V: now also C24.1, C25.1, C26.1
- net +5V: now also IC2.AVCC, IC8.+5V, JP2.2, JP3.1
- net E_RESET: now also IC2.PB1(OC1A)
- net GND: now also C23.2, IC2.GND, IC8.GND, JP2.1, JP3.2
- net GND1: now also C24.2, C25.2, C26.2
- net I_CONTRAST: now also JP2.3
- net I_E: now also IC6.P4; no longer IC6.P5
- net I_RS: now also IC6.P6; no longer IC6.P7
- net I_RW: now also IC6.P5; no longer IC6.P6
- net RESET: now also IC8./RST
- net SD_DETECT: now also IC2.PD7(AIN1)
- net SD_SELECT: now also IC2.PB0(ICP); no longer IC2.PB1(OC1A)
- net SPI0: now also IC2.ADC6
Other:
- moved on the sheet: G1, IC1, JP4, Q5, R10, R11, X4-1, X4-2, X6-1, X6-2, X6-3, X6-4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

Commit message: Prepared to rezonver
Parts:
- removed Q5: (no value), MyLib:MA306
- removed U$1, U$2, U$3, U$5, U$6, U$7, U$8: NSI45020AT1GSOD-123, MyLib:NSI45020AT1GSOD-123
- removed U$10: 2X16LCDBOTH, MyLib:2X16LCDBOTH
- added D15, D16, D18, D19, D20, D21: BAV199, MyLib:BAV199
- added D17: CDSOT23-SM712SOT23-R, MyLib:CDSOT23-SM712SOT23-R
- added JP5: (no value), pinhead:PINHD-1X3
- added LCD1: 2X16LCDBOTHM162SD07, MyLib:2X16LCDBOTHM162SD07
- added Q1: (no value), crystal:CRYSTALSM49
- C1, C2, C4: value (none) -> 0.1; device rcl:CPOL-EU153CLV-0605 -> rcl:C-EUC0805
- C11, C12: value (none) -> 0.1
- C13: value 10uF -> 0.1
- C14, C16: value 100nF -> 0.1
- C15: value 10nF -> (none); device rcl:C-EUC0805 -> rcl:CPOL-EU153CLV-0605
- C17: value 10nF -> (none)
- C18: value 100nF -> (none)
- C19: value 100nF -> 10uF
- C20: value 10uF -> 100nF
- C21, C23, C25: value 0.1 -> 100nF
- C22, C24: value 0.1 -> 10nF
- C26: value 0.1 -> 10uF
- C6, C9: value 0.1 -> (none); device rcl:C-EUC0805 -> rcl:CPOL-EU153CLV-0605
- D1, D2, D4, D5, D6, D7, D8: value BAV199 -> NSI45020AT1GSOD-123; device MyLib:BAV199 -> MyLib:NSI45020AT1GSOD-123
- D11: value CDSOT23-SM712SOT23-R -> BAV199; device MyLib:CDSOT23-SM712SOT23-R -> MyLib:BAV199
- IC1: value DS1307Z -> LM1117IMPX-3.3; device MyLib:DS1307Z -> lm1117:LM1117IMPX-3.3
- IC2: value MEGA8-AI -> DS1813-SMD; device atmel:MEGA8-AI -> MyLib:DS1813-SMD
- IC3: value LM1117IMPX-3.3 -> PCF8574T; device lm1117:LM1117IMPX-3.3 -> micro-philips:PCF8574T
- IC4: value PCF8574T -> MEGA8-AI; device micro-philips:PCF8574T -> atmel:MEGA8-AI
- IC5: value PCF8574T -> DS1307Z; device micro-philips:PCF8574T -> MyLib:DS1307Z
- IC8: value DS1813-SMD -> PCF8574T; device MyLib:DS1813-SMD -> micro-philips:PCF8574T
- JP1: device pinhead:PINHD-1X9 -> pinhead:PINHD-2X3
- JP2: device pinhead:PINHD-1X3 -> pinhead:PINHD-1X4
- JP3: device pinhead:PINHD-1X4 -> pinhead:PINHD-1X2
- JP4: device pinhead:PINHD-2X3 -> pinhead:PINHD-1X9
- Q2: device crystal:CRYSTALSM49 -> MyLib:MA306
- R10: value 3k3 -> 50
- R12: value 3.3k -> 100k
- R13: value 100k -> 3k3; device rcl:R-EU_M0805 -> rcl:R-EU_R0805
- R3: value 50 -> 1.8k; device rcl:R-EU_R0805 -> rcl:R-EU_M0805
- R4: value 50 -> 3.3k; device rcl:R-EU_R0805 -> rcl:R-EU_M0805
- R5: value 3.3k -> 1.8k
- R8: value 1.8k -> 3.3k
- R9: value 1.8k -> 50; device rcl:R-EU_M0805 -> rcl:R-EU_R0805
- U1: value ADM2587EBRWZ -> TRACO_TEL_5-1211; device Analog Devices_By_element14_Batch_1:ADM2587EBRWZ -> MyLib:TRACO_TEL_5-1211
- U2: value TRACO_TEL_5-1211 -> ADM2587EBRWZ; device MyLib:TRACO_TEL_5-1211 -> Analog Devices_By_element14_Batch_1:ADM2587EBRWZ
- X1: value MKDSN1,5/3-5,08 -> MKDSN1,5/2-5,08; device MyLib:MKDSN1,5/3-5,08 -> con-phoenix-508:MKDSN1,5/2-5,08
- X2: value MKDSN1,5/4-5,08 -> 22-23-2021; device con-phoenix-508:MKDSN1,5/4-5,08 -> con-molex:22-23-2021
- X4: value MKDSN1,5/2-5,08 -> MKDSN1,5/4-5,08; device con-phoenix-508:MKDSN1,5/2-5,08 -> con-phoenix-508:MKDSN1,5/4-5,08
- X5: value 22-23-2021 -> 22-23-2051; device con-molex:22-23-2021 -> con-molex:22-23-2051
- X6: value 22-23-2051 -> 22-23-2041; device con-molex:22-23-2051 -> con-molex:22-23-2041
- X7: value 22-23-2041 -> MKDSN1,5/4-5,08; device con-molex:22-23-2041 -> con-phoenix-508:MKDSN1,5/4-5,08
- X8: value MKDSN1,5/4-5,08 -> MKDSN1,5/3-5,08; device con-phoenix-508:MKDSN1,5/4-5,08 -> MyLib:MKDSN1,5/3-5,08
- renumbered R15 to R14, U$11 to D22, U$12 to D23, U$13 to D24, U$14 to D25, U$4 to D3, U$9 to MOD1
Connections:
- removed net INT-S: IC4.P0
- new net N$68: JP3.2, R11.2, R13.2
- net +24V: now also C1.1, C2.1, C4.1, C7.1, C9.+, D11.C, D15.C, D16.C, D18.C, D19.C, D20.C, D21.C, OC11.COL, OC12.COL, U1.+VIN@1, U1.+VIN@2, X1-1.KL; no longer C24.1, C25.1, C26.1, C4.+, C6.1, D1.C, D2.C, D4.C, D5.C, D6.C, D7.C, D8.C, OC7.COL, OC8.COL, U2.+VIN@1, U2.+VIN@2, X4-1.KL
- net +3V3: now also C13.1, C14.1, C15.+, IC1.OUT, IC1.OUT1, R12.2; no longer C1.+, C5.1, C7.1, IC3.OUT, IC3.OUT1, R13.2
- net +5V: now also C11.1, C12.1, C5.1, C6.+, IC1.IN, IC2.+5V, IC3.A0, IC3.VDD, IC4.AVCC, IC4.VCC@1, IC4.VCC@2, IC5.VCC, IC8.A0, IC8.A1, IC8.VDD, JP1.2, JP2.1, JP5.2, LCD1.VDD, U1.+VOUT, U2.VCC, U2.VCC_2, X2-1.S, X6-1.S; no longer C17.1, C18.1, C2.+, C9.1, IC1.VCC, IC2.AVCC, IC2.VCC@1, IC2.VCC@2, IC3.IN, IC4.VDD, IC5.A0, IC5.VDD, IC6.A1, IC7.A0, IC8.+5V, JP2.2, JP4.2, R10.2, R11.2, U$10.VDD, U1.VCC, U1.VCC_2, U2.+VOUT, X5-1.S, X7-1.S
- net 485_R/W: now also IC4.PD4(XCK/T0), U2.DE, U2.~RE; no longer IC2.PD4(XCK/T0), U1.DE, U1.~RE
- net A: now also D17.P$1, U2.A; no longer D11.P$1, U1.A
- net B: now also D17.P$2, U2.B; no longer D11.P$2, U1.B
- net E_RESET: now also IC4.PB1(OC1A); no longer IC2.PB1(OC1A)
- net E_SELECT: now also IC4.PB2(SS/OC1B); no longer IC2.PB2(SS/OC1B)
- net GND: now also C12.2, C13.2, C14.2, C15.-, C16.2, C17.1, C6.-, IC3.A1, IC3.A2, IC3.VSS, IC4.GND, IC4.GND@1, IC4.GND@2, IC5.GND, IC6.A1, IC7.A0, IC8.A2, IC8.VSS, JP1.6, JP2.2, JP4.1, JP5.1, LCD1.VSS, MOD1.GND@2, OC11.C, OC12.C, OC7.EMIT, OC8.EMIT, R4.1, R8.1, U1.-V0UT, U2.GND1, U2.GND1_2, U2.GND1_3, U2.GND1_4, X2-2.S, X5-5.S, X6-4.S; no longer C1.-, C12.1, C17.2, C2.-, C23.2, C7.2, C9.2, IC2.GND@1, IC2.GND@2, IC3.GND, IC4.A0, IC4.A1, IC4.A2, IC4.VSS, IC5.A1, IC5.A2, IC5.VSS, IC8.GND, JP1.1, JP2.1, JP3.2, JP4.6, OC11.EMIT, OC12.EMIT, OC7.C, OC8.C, R12.1, R5.1, U$10.VSS, U1.GND1, U1.GND1_2, U1.GND1_3, U1.GND1_4, U2.-V0UT, X5-2.S, X6-5.S, X7-4.S
- net GND1: now also C1.2, C2.2, C23.2, C4.2, C7.2, C9.-, D11.A, D15.A, D16.A, D17.P$3, D18.A, D19.A, D20.A, D21.A, OC7.C, OC8.C, U1.-VIN@1, U1.-VIN@2, U2.GND2, U2.GND2_2, X8-2.KL; no longer C13.2, C15.2, C16.2, C25.2, C4.-, C6.2, D1.A, D11.P$3, D2.A, D4.A, D5.A, D6.A, D7.A, D8.A, OC11.C, OC12.C, U1.GND2, U1.GND2_2, U2.-VIN@1, U2.-VIN@2, X4-2.KL
- net INT0: now also IC4.PD2(INT0), IC6.!INT; no longer IC2.PD2(INT0), IC4.!INT
- net INT1: now also IC3.!INT, IC4.PD3(INT1); no longer IC2.PD3(INT1), IC5.!INT
- net I_CONTRAST: now also JP5.3, LCD1.VO; no longer JP2.3, U$10.VO
- net I_D0: now also IC8.P0, LCD1.D0; no longer IC7.P0, U$10.D0
- net I_D1: now also IC8.P1, LCD1.D1; no longer IC7.P1, U$10.D1
- net I_D2: now also IC8.P2, LCD1.D2; no longer IC7.P2, U$10.D2
- net I_D3: now also IC8.P3, LCD1.D3; no longer IC7.P3, U$10.D3
- net I_D4: now also IC8.P4, LCD1.D4; no longer IC7.P4, U$10.D4
- net I_D5: now also IC8.P5, LCD1.D5; no longer IC7.P5, U$10.D5
- net I_D6: now also IC8.P6, LCD1.D6; no longer IC7.P6, U$10.D6
- net I_D7: now also IC8.P7, LCD1.D7; no longer IC7.P7, U$10.D7
- net I_E: now also IC7.P4, LCD1.E; no longer IC6.P4, U$10.E
- net I_RS: now also IC7.P6, LCD1.RS; no longer IC6.P6, U$10.RS
- net I_RW: now also IC7.P5, LCD1.RW; no longer IC6.P5, U$10.RW
- net MISO: now also IC4.PB4(MISO), JP1.1, X5-2.S; no longer IC2.PB4(MISO), JP4.1, X6-2.S
- net MOSI: now also IC4.PB3(MOSI/OC2), JP1.4, R5.2, X5-3.S; no longer IC2.PB3(MOSI/OC2), JP4.4, R8.2, X6-3.S
- net N$1: now also X8-1.KL; no longer X1-1.KL
- net N$10: now also D18.AC, OC12.EMIT; no longer D13.AC, OC10.EMIT
- net N$11: now also D19.AC, OC11.EMIT; no longer D4.AC, OC9.EMIT
- net N$12: now also D20.AC, OC10.EMIT; no longer D1.AC, OC8.EMIT
- net N$13: now also D21.AC, OC9.EMIT; no longer D2.AC, OC7.EMIT
- net N$14: now also C18.1, IC4.PB7(XTAL2/TOSC2), Q1.1; no longer C11.1, IC2.PB7(XTAL2/TOSC2), Q2.1
- net N$15: now also OC9.A; no longer OC7.A
- net N$16: now also D1.C, D9.AC; no longer D14.AC, U$1.C
- net N$17: now also D10.AC, D2.C; no longer D5.AC, U$2.C
- net N$18: now also OC10.A; no longer OC8.A
- net N$19: now also OC11.A, R9.1; no longer OC9.A, R3.1
- net N$2: now also X8-3.KL; no longer X1-3.KL
- net N$20: now also IC5.VBAT; no longer IC1.VBAT
- net N$21: now also D1.A, X4-1.KL; no longer U$1.A, X2-1.KL
- net N$22: now also D2.A, X4-2.KL; no longer U$2.A, X2-2.KL
- net N$23: now also IC5.X1, Q2.1; no longer IC1.X1, Q5.1
- net N$24: now also D11.AC; no longer D6.AC
- net N$25: now also IC5.X2, Q2.2; no longer IC1.X2, Q5.2
- net N$26: now also C17.2, IC4.PB6(XTAL1/TOSC1), Q1.2; no longer C12.2, IC2.PB6(XTAL1/TOSC1), Q2.2
- net N$27: now also D12.AC, D4.C; no longer D7.AC, U$5.C
- net N$28: now also D7.A, X3-3.KL; no longer U$3.A, X8-3.KL
- net N$29: now also OC12.A, R10.1; no longer OC10.A, R4.1
- net N$3: now also C23.1, C24.1, C26.1, U2.VISOIN; no longer C13.1, C15.1, C16.1, U1.VISOIN
- net N$30: now also D13.AC, D5.C; no longer D8.AC, U$6.C
- net N$32: now also D14.AC, D6.C; no longer D9.AC, U$7.C
- net N$33: now also D4.A, X4-4.KL; no longer U$5.A, X2-4.KL
- net N$34: now also D15.AC, D7.C, OC7.A; no longer D10.AC, OC11.A, U$3.C
- net N$35: now also X4-3.KL; no longer X2-3.KL
- net N$36: now also D16.AC, D8.C, OC8.A; no longer D12.AC, OC12.A, U$8.C
- net N$37: now also D5.A, X3-1.KL; no longer U$6.A, X8-1.KL
- net N$38: now also D6.A, X3-2.KL; no longer U$7.A, X8-2.KL
- net N$39: now also D8.A, X3-4.KL; no longer U$8.A, X8-4.KL
- net N$4: now also C25.2, U2.GND2_3, U2.GND2_4; no longer C14.2, U1.GND2_3, U1.GND2_4
- net N$40: now also IC3.P2; no longer IC5.P2
- net N$41: now also IC3.P1, OC7.COL; no longer IC5.P1, OC11.COL
- net N$42: now also IC3.P0, OC8.COL; no longer IC5.P0, OC12.COL
- net N$43: now also R7.1, R8.2; no longer R12.2, R9.1
- net N$45: now also IC6.P7, JP4.2; no longer IC4.P7, JP1.2
- net N$46: now also IC6.P6, JP4.3; no longer IC4.P6, JP1.3
- net N$47: now also IC6.P5, JP4.4; no longer IC4.P5, JP1.4
- net N$48: now also IC6.P1, JP4.6; no longer IC4.P1, JP1.6
- net N$49: now also IC6.P4, JP4.5; no longer IC4.P4, JP1.5
- net N$5: now also C25.1, U2.VISOOUT; no longer C14.1, U1.VISOOUT
- net N$50: now also IC6.P3, JP4.9; no longer IC4.P3, JP1.9
- net N$51: now also IC6.P2, JP4.7; no longer IC4.P2, JP1.7
- net N$53: now also JP4.8; no longer JP1.8
- net N$54: now also IC3.P7; no longer IC5.P7
- net N$55: now also IC3.P6; no longer IC5.P6
- net N$56: now also IC3.P5; no longer IC5.P5
- net N$57: now also IC3.P4; no longer IC5.P4
- net N$58: now also IC3.P3; no longer IC5.P3
- net N$59: now also R5.1; no longer R8.1
- net N$6: now also IC4.PC0(ADC0), R10.2; no longer IC2.PC0(ADC0), R4.2
- net N$60: now also R3.1, R4.2; no longer R5.2, R7.1
- net N$61: now also C16.1, IC4.AREF; no longer C23.1, IC2.AREF
- net N$62: now also X7-1.KL; no longer X3-1.KL
- net N$63: now also X7-2.KL; no longer X3-2.KL
- net N$64: now also IC4.PD6(AIN0), JP2.3; no longer IC2.PD6(AIN0), JP3.3
- net N$65: now also X7-3.KL; no longer X3-3.KL
- net N$66: now also IC4.PD5(T1), JP2.4; no longer IC2.PD5(T1), JP3.4
- net N$67: now also X7-4.KL; no longer X3-4.KL
- net N$7: now also IC4.PC1(ADC1), R9.2; no longer IC2.PC1(ADC1), R3.2
- net N$8: now also IC4.PC2(ADC2); no longer IC2.PC2(ADC2)
- net N$9: now also IC4.PC3(ADC3); no longer IC2.PC3(ADC3)
- net RESET: now also IC2./RST, IC4.PC6(/RESET), JP1.5; no longer IC2.PC6(/RESET), IC8./RST, JP4.5
- net RXD: now also IC4.PD0(RXD), U2.RXD; no longer IC2.PD0(RXD), U1.RXD
- net SCK: now also IC4.PB5(SCK), JP1.3, R3.2, X5-1.S; no longer IC2.PB5(SCK), JP4.3, R7.2, X6-1.S
- net SCL: now also IC3.SCL, IC4.PC5(ADC5/SCL), IC8.SCL, R11.1, X6-3.S; no longer IC1.SCL, IC2.PC5(ADC5/SCL), IC4.SCL, R10.1, X7-3.S
- net SDA: now also IC3.SDA, IC4.PC4(ADC4/SDA), IC8.SDA, R13.1, X6-2.S; no longer IC1.SDA, IC2.PC4(ADC4/SDA), IC4.SDA, R11.1, X7-2.S
- net SD_DETECT: now also IC4.PD7(AIN1), R12.1; no longer IC2.PD7(AIN1), R13.1
- net SD_SELECT: now also IC4.PB0(ICP), R7.2; no longer IC2.PB0(ICP), R9.2
- net SPI0: now also IC4.ADC6, X5-4.S; no longer IC2.ADC6, X6-4.S
- net TXD: now also IC4.PD1(TXD), U2.TXD; no longer IC2.PD1(TXD), U1.TXD
Other:
- moved on the sheet: C10, C11, C12, C13, C14, C16, C17, C18, C19, C20, C21, C22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

Commit message: wip
Parts:
- R11, R13: value 3k3 -> 10k
Connections:
- net A renamed A-
- net B renamed B+
- new net Y: U2.Y
- new net Z: U2.Z
Changed lines of the file:
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@@
 <part name="GND28" library="supply1" deviceset="GND" device=""/>
 <part name="GND32" library="supply1" deviceset="GND" device=""/>
-<part name="R11" library="rcl" deviceset="R-EU_" device="R0805" value="3k3"/>
-<part name="R13" library="rcl" deviceset="R-EU_" device="R0805" value="3k3"/>
+<part name="R11" library="rcl" deviceset="R-EU_" device="R0805" value="10k"/>
+<part name="R13" library="rcl" deviceset="R-EU_" device="R0805" value="10k"/>
 <part name="X6" library="con-molex" deviceset="22-23-2041" device=""/>
 <part name="GND37" library="supply1" deviceset="GND" device=""/>
@@
 </segment>
 </net>
-<net name="B" class="0">
+<net name="B+" class="0">
 <segment>
 <pinref part="Z2" gate="G$1" pin="2"/>
@@
 </segment>
 </net>
-<net name="A" class="0">
+<net name="A-" class="0">
 <segment>
 <pinref part="D17" gate="G$1" pin="P$1"/>
@@
 </segment>
 </net>
+<net name="Y" class="0">
+<segment>
+<pinref part="U2" gate="A" pin="Y"/>
+<wire x1="251.46" y1="243.84" x2="297.18" y2="243.84" width="0.1524" layer="91"/>
+<label x="287.02" y="243.84" size="1.778" layer="95"/>
+</segment>
+</net>
+<net name="Z" class="0">
+<segment>
+<pinref part="U2" gate="A" pin="Z"/>
+<wire x1="251.46" y1="241.3" x2="297.18" y2="241.3" width="0.1524" layer="91"/>
+<label x="287.02" y="241.3" size="1.778" layer="95"/>
+</segment>
+</net>
